File: Design/Rapid_Core-RCP.kicad_pcb (KiCad board)
At the start: 0 parts

Commit message: Schematic Design complete
Parts:
- added C1: 10uF, Capacitor_SMD:C_0805_2012Metric_Pad1.18x1.45mm_HandSolder, F.Cu at (118.2, 102.8)
- added C10: 0u1F, Capacitor_SMD:C_0603_1608Metric_Pad1.08x0.95mm_HandSolder, F.Cu at (150.2, 107.6)
- added C11: 15pf, Capacitor_SMD:C_0603_1608Metric, F.Cu at (145.4, 130.0)
- added C12: 15pF, Capacitor_SMD:C_0603_1608Metric, F.Cu at (145.4, 132.5)
- added C13: 0u1F, Capacitor_SMD:C_0603_1608Metric_Pad1.08x0.95mm_HandSolder, F.Cu at (150.2, 110.1)
- added C14: 10uf, Capacitor_SMD:C_0805_2012Metric_Pad1.18x1.45mm_HandSolder, F.Cu at (118.2, 117.9)
- added C15: 1uf, Capacitor_SMD:C_0603_1608Metric_Pad1.08x0.95mm_HandSolder, F.Cu at (150.2, 112.6)
- added C16: 0.1uf, Capacitor_SMD:C_0603_1608Metric_Pad1.08x0.95mm_HandSolder, F.Cu at (150.2, 115.1)
- added C17: 4.7uf 6.3V XR7, Capacitor_SMD:C_0805_2012Metric_Pad1.18x1.45mm_HandSolder, F.Cu at (118.2, 120.9)
- added C18: 0.1uf, Capacitor_SMD:C_0603_1608Metric_Pad1.08x0.95mm_HandSolder, F.Cu at (150.2, 117.6)
- added C19: 10uf, Capacitor_SMD:C_0805_2012Metric_Pad1.18x1.45mm_HandSolder, F.Cu at (118.2, 123.9)
- added C2: 0u1F, Capacitor_SMD:C_0603_1608Metric_Pad1.08x0.95mm_HandSolder, F.Cu at (150.2, 102.6)
- added C20: 1uf, Capacitor_SMD:C_0603_1608Metric_Pad1.08x0.95mm_HandSolder, F.Cu at (154.5, 102.6)
- added C21: 0.1uf, Capacitor_SMD:C_0603_1608Metric_Pad1.08x0.95mm_HandSolder, F.Cu at (154.5, 105.1)
- added C22: 0.1uf, Capacitor_SMD:C_0603_1608Metric_Pad1.08x0.95mm_HandSolder, F.Cu at (154.5, 107.6)
- added C23: 0.1uf, Capacitor_SMD:C_0603_1608Metric_Pad1.08x0.95mm_HandSolder, F.Cu at (154.5, 110.1)
- added C24: 0.1uf, Capacitor_SMD:C_0603_1608Metric_Pad1.08x0.95mm_HandSolder, F.Cu at (154.5, 112.6)
- added C25: 10uf, Capacitor_SMD:C_0805_2012Metric_Pad1.18x1.45mm_HandSolder, F.Cu at (161.2, 33.8)
- added C26: 1uf, Capacitor_SMD:C_0603_1608Metric_Pad1.08x0.95mm_HandSolder, F.Cu at (143.6, 33.6)
- added C27: 0.1uf, Capacitor_SMD:C_0603_1608Metric_Pad1.08x0.95mm_HandSolder, F.Cu at (143.6, 36.1)
- added C28: 0.1uf, Capacitor_SMD:C_0603_1608Metric_Pad1.08x0.95mm_HandSolder, F.Cu at (143.6, 38.6)
- added C29: 1uf, Capacitor_SMD:C_0603_1608Metric_Pad1.08x0.95mm_HandSolder, F.Cu at (143.6, 41.1)
- added C3: 220uF, Capacitor_SMD:C_0805_2012Metric_Pad1.18x1.45mm_HandSolder, F.Cu at (118.2, 105.8)
- added C30: 0.1uf, Capacitor_SMD:C_0603_1608Metric_Pad1.08x0.95mm_HandSolder, F.Cu at (143.6, 43.6)
- added C31: 10uf, Capacitor_SMD:C_0805_2012Metric_Pad1.18x1.45mm_HandSolder, F.Cu at (161.2, 36.8)
- added C32: 1uf, Capacitor_SMD:C_0603_1608Metric_Pad1.08x0.95mm_HandSolder, F.Cu at (143.6, 46.1)
- added C33: 10uf, Capacitor_SMD:C_0805_2012Metric_Pad1.18x1.45mm_HandSolder, F.Cu at (161.2, 39.8)
- added C34: 10uf, Capacitor_SMD:C_0805_2012Metric_Pad1.18x1.45mm_HandSolder, F.Cu at (161.2, 42.9)
- added C35: 1uf, Capacitor_SMD:C_0603_1608Metric_Pad1.08x0.95mm_HandSolder, F.Cu at (143.6, 48.6)
- added C36: 0.1uf, Capacitor_SMD:C_0603_1608Metric_Pad1.08x0.95mm_HandSolder, F.Cu at (143.6, 51.1)
- added C37: 0.1uf, Capacitor_SMD:C_0603_1608Metric_Pad1.08x0.95mm_HandSolder, F.Cu at (143.6, 53.6)
- added C38: 0.1uf, Capacitor_SMD:C_0603_1608Metric_Pad1.08x0.95mm_HandSolder, F.Cu at (143.6, 56.2)
- added C39: 1uf, Capacitor_SMD:C_0603_1608Metric_Pad1.08x0.95mm_HandSolder, F.Cu at (147.9, 33.6)
- added C4: 220uF, Capacitor_SMD:C_0805_2012Metric_Pad1.18x1.45mm_HandSolder, F.Cu at (118.2, 108.8)
- added C40: 1uf, Capacitor_SMD:C_0603_1608Metric_Pad1.08x0.95mm_HandSolder, F.Cu at (147.9, 36.1)
- added C41: 10uf, Capacitor_SMD:C_0805_2012Metric_Pad1.18x1.45mm_HandSolder, F.Cu at (161.2, 45.9)
- added C42: 10uf, Capacitor_SMD:C_0805_2012Metric_Pad1.18x1.45mm_HandSolder, F.Cu at (161.2, 48.9)
- added C43: 10uf, Capacitor_SMD:C_0805_2012Metric_Pad1.18x1.45mm_HandSolder, F.Cu at (161.2, 51.9)
- added C44: 1uf, Capacitor_SMD:C_0603_1608Metric_Pad1.08x0.95mm_HandSolder, F.Cu at (147.9, 38.6)
- added C45: 0.1uf, Capacitor_SMD:C_0603_1608Metric_Pad1.08x0.95mm_HandSolder, F.Cu at (147.9, 41.1)
- added C46: 10uf, Capacitor_SMD:C_0805_2012Metric_Pad1.18x1.45mm_HandSolder, F.Cu at (161.2, 54.9)
- added C47: 1uf, Capacitor_SMD:C_0603_1608Metric_Pad1.08x0.95mm_HandSolder, F.Cu at (147.9, 43.6)
- added C48: 0.1uf, Capacitor_SMD:C_0603_1608Metric_Pad1.08x0.95mm_HandSolder, F.Cu at (147.9, 46.1)
- added C49: 4u7F 1mOhm, Capacitor_SMD:C_0805_2012Metric_Pad1.18x1.45mm_HandSolder, F.Cu at (193.6, 110.2)
- added C5: 20pF, Capacitor_SMD:C_0603_1608Metric, F.Cu at (145.4, 125.0)
- added C50: 66uF LDO, Capacitor_SMD:CP_Elec_5x5.8, F.Cu at (174.3, 117.7)
- added C51: 0.22uF 1m, Capacitor_SMD:C_0603_1608Metric_Pad1.08x0.95mm_HandSolder, F.Cu at (167.7, 107.1)
- added C52: 0.22uF 1m, Capacitor_SMD:C_0603_1608Metric_Pad1.08x0.95mm_HandSolder, F.Cu at (167.7, 109.6)
- added C53: 1uF 6.065m, Capacitor_SMD:C_0603_1608Metric_Pad1.08x0.95mm_HandSolder, F.Cu at (167.7, 112.1)
- added C54: 1uF 6.065m, Capacitor_SMD:C_0603_1608Metric_Pad1.08x0.95mm_HandSolder, F.Cu at (167.7, 114.7)
- added C55: 33uF LDO, Capacitor_SMD:CP_Elec_4x5.8, F.Cu at (198.5, 98.4)
- added C56: 0.1uF 1m, Capacitor_SMD:C_0603_1608Metric_Pad1.08x0.95mm_HandSolder, F.Cu at (167.7, 117.2)
- added C57: 27pF 1mohm, Capacitor_SMD:C_0805_2012Metric_Pad1.18x1.45mm_HandSolder, F.Cu at (193.6, 113.2)
- added C58: 100uF 1mohm, Capacitor_SMD:C_0805_2012Metric_Pad1.18x1.45mm_HandSolder, F.Cu at (193.6, 116.2)
- added C59: 100uF 1mohm, Capacitor_SMD:C_0805_2012Metric_Pad1.18x1.45mm_HandSolder, F.Cu at (193.6, 119.2)
- added C6: 20pF, Capacitor_SMD:C_0603_1608Metric, F.Cu at (145.4, 127.5)
- added C60: 100uF 30mohm, Capacitor_SMD:C_0805_2012Metric_Pad1.18x1.45mm_HandSolder, F.Cu at (193.6, 122.2)
- added C62: 4700pF, Capacitor_SMD:C_0603_1608Metric_Pad1.08x0.95mm_HandSolder, F.Cu at (147.9, 48.6)
- added C7: 10uF, Capacitor_SMD:C_0805_2012Metric_Pad1.18x1.45mm_HandSolder, F.Cu at (118.2, 111.8)
- added C8: 0u1F, Capacitor_SMD:C_0603_1608Metric_Pad1.08x0.95mm_HandSolder, F.Cu at (150.2, 105.1)
- added C9: 10uF, Capacitor_SMD:C_0805_2012Metric_Pad1.18x1.45mm_HandSolder, F.Cu at (118.2, 114.9)
- added D1: D, Diode_SMD:D_SOD-323_HandSoldering, F.Cu at (134.4, 126.5)
- added D2: D, Diode_SMD:D_SOD-323_HandSoldering, F.Cu at (134.4, 129.5)
- added D3: RED, LED_SMD:LED_0603_1608Metric_Pad1.05x0.95mm_HandSolder, F.Cu at (140.8, 126.2)
- added D4: RED, LED_SMD:LED_0603_1608Metric_Pad1.05x0.95mm_HandSolder, F.Cu at (140.8, 128.8)
- added D5: SM712_SOT23, Package_TO_SOT_SMD:SOT-23, F.Cu at (165.5, 59.6)
- added D6: SM712_SOT23, Package_TO_SOT_SMD:SOT-23, F.Cu at (165.5, 64.1)
- added D7: SM712_SOT23, Package_TO_SOT_SMD:SOT-23, F.Cu at (165.5, 68.5)
- added D8: SM712_SOT23, Package_TO_SOT_SMD:SOT-23, F.Cu at (165.5, 73.0)
- added D9: RED, LED_SMD:LED_0603_1608Metric_Pad1.05x0.95mm_HandSolder, F.Cu at (181.4, 121.8)
- added FB1: FerriteBead, Inductor_SMD:L_0805_2012Metric_Pad1.05x1.20mm_HandSolder, F.Cu at (134.2, 132.3)
- added FID1: Fiducial, Fiducial:Fiducial_1.5mm_Mask3mm, F.Cu at (118.1, 85.4)
- added FID2: Fiducial, Fiducial:Fiducial_1.5mm_Mask3mm, F.Cu at (118.1, 89.9)
- added FID3: Fiducial, Fiducial:Fiducial_1.5mm_Mask3mm, F.Cu at (118.1, 94.5)
- added FID4: Fiducial, Fiducial:Fiducial_1.5mm_Mask3mm, F.Cu at (118.1, 99.0)
- added H1: MountingHole_Pad, MountingHole:MountingHole_2.2mm_M2_Pad, F.Cu at (123.6, 104.3)
- added H2: MountingHole_Pad, MountingHole:MountingHole_2.2mm_M2_Pad, F.Cu at (123.6, 110.2)
- added H3: MountingHole_Pad, MountingHole:MountingHole_2.2mm_M2_Pad, F.Cu at (123.6, 116.2)
- added H4: MountingHole_Pad, MountingHole:MountingHole_2.2mm_M2_Pad, F.Cu at (123.6, 122.1)
- added IC1: TLIN1039DDFRQ1, TLIN1039DDFRQ1:SOT65P280X110-8N, F.Cu at (129.2, 127.3)
- added IC2: TLIN1039DDFRQ1, TLIN1039DDFRQ1:SOT65P280X110-8N, F.Cu at (129.2, 131.8)
- added IC3: SHT30A-DIS-B2.5KS, SHT30A-DIS-B2.5KS:SON50P250X250X100-9N-D, F.Cu at (123.0, 127.2)
- added IC4: LM60440ARPKR, LM60440ARPKR_Buck:LM60440AQRPKRQ1, F.Cu at (197.1, 104.0)
- added J1: CMD PIN, Connector_PinHeader_2.54mm:PinHeader_1x02_P2.54mm_Vertical, F.Cu at (155.0, 126.4)
- added J10: CAN-1, TerminalBlock_Phoenix:TerminalBlock_Phoenix_MKDS-1,5-2_1x02_P5.00mm_Horizontal, F.Cu at (238.8, 36.8)
- added J11: RS-485_1, TerminalBlock_Phoenix:TerminalBlock_Phoenix_MKDS-1,5-2_1x02_P5.00mm_Horizontal, F.Cu at (238.8, 48.6)
- added J12: RS-485_2, TerminalBlock_Phoenix:TerminalBlock_Phoenix_MKDS-1,5-2_1x02_P5.00mm_Horizontal, F.Cu at (238.8, 71.1)
- added J14: CAN-2, TerminalBlock_Phoenix:TerminalBlock_Phoenix_MKDS-1,5-2_1x02_P5.00mm_Horizontal, F.Cu at (251.5, 71.1)
- added J15: Input Power, TerminalBlock_Phoenix:TerminalBlock_Phoenix_MKDS-1,5-2_1x02_P5.00mm_Horizontal, F.Cu at (182.7, 114.9)
- added J2: CMD PIN, Connector_PinHeader_2.54mm:PinHeader_1x02_P2.54mm_Vertical, F.Cu at (159.6, 126.4)
- added J3: LIN_1, TerminalBlock_Phoenix:TerminalBlock_Phoenix_MKDS-1,5-2_1x02_P5.00mm_Horizontal, F.Cu at (130.1, 107.5)
- added J4: LIN_2, TerminalBlock_Phoenix:TerminalBlock_Phoenix_MKDS-1,5-2_1x02_P5.00mm_Horizontal, F.Cu at (130.1, 119.4)
- added J5: GPIO_CONN_x_4, Connector_PinHeader_2.54mm:PinHeader_1x08_P2.54mm_Vertical, F.Cu at (145.7, 103.6)
- added J6: SWD_Debug, Connector_PinHeader_2.54mm:PinHeader_1x05_P2.54mm_Vertical, F.Cu at (150.3, 121.2)
- added J7: SPI_CONN, Connector_PinHeader_2.54mm:PinHeader_1x10_P2.54mm_Vertical, F.Cu at (113.5, 85.4)
- added J8: USART, Connector_PinHeader_2.54mm:PinHeader_1x04_P2.54mm_Vertical, F.Cu at (159.9, 85.4)
- added L1: 51uH 0.2A 1R, ACT45B-510-2P-TL003:IND_ACT45R_TDK, F.Cu at (159.3, 59.9)
- added L2: 51uH 0.2A 1R, ACT45B-510-2P-TL003:IND_ACT45R_TDK, F.Cu at (159.3, 65.0)
- added L3: 51uH 0.2A 1R, ACT45B-510-2P-TL003:IND_ACT45R_TDK, F.Cu at (159.3, 70.1)
- added L4: 51u 0.2A 1R, ACT45B-510-2P-TL003:IND_ACT45R_TDK, F.Cu at (159.3, 75.1)
- added L5: 8.2 24mohm, Inductor_SMD:L_Coilcraft_XAL6060-XXX, F.Cu at (174.0, 110.1)
- added R1: 10K, Resistor_SMD:R_0805_2012Metric_Pad1.20x1.40mm_HandSolder, F.Cu at (141.0, 102.8)
- added R10: 10k, Resistor_SMD:R_0805_2012Metric_Pad1.20x1.40mm_HandSolder, F.Cu at (141.0, 123.4)
- added R11: 0, Resistor_SMD:R_0603_1608Metric_Pad0.98x0.95mm_HandSolder, F.Cu at (158.9, 102.6)
- added R12: 0, Resistor_SMD:R_0603_1608Metric_Pad0.98x0.95mm_HandSolder, F.Cu at (158.9, 105.1)
- added R13: 0, Resistor_SMD:R_0603_1608Metric_Pad0.98x0.95mm_HandSolder, F.Cu at (158.9, 107.6)
- added R14: 0, Resistor_SMD:R_0603_1608Metric_Pad0.98x0.95mm_HandSolder, F.Cu at (158.9, 110.1)
- added R15: 0 C, Resistor_SMD:R_0603_1608Metric_Pad0.98x0.95mm_HandSolder, F.Cu at (147.9, 51.1)
- added R16: 0 C, Resistor_SMD:R_0603_1608Metric_Pad0.98x0.95mm_HandSolder, F.Cu at (147.9, 53.6)
- added R17: 0 RS, Resistor_SMD:R_0603_1608Metric_Pad0.98x0.95mm_HandSolder, F.Cu at (147.9, 56.2)
- added R18: 0 RS, Resistor_SMD:R_0603_1608Metric_Pad0.98x0.95mm_HandSolder, F.Cu at (152.3, 33.6)
- added R19: 0 RS, Resistor_SMD:R_0603_1608Metric_Pad0.98x0.95mm_HandSolder, F.Cu at (152.3, 36.1)
- added R2: 10K, Resistor_SMD:R_0805_2012Metric_Pad1.20x1.40mm_HandSolder, F.Cu at (141.0, 105.7)
- added R20: 0 RS, Resistor_SMD:R_0603_1608Metric_Pad0.98x0.95mm_HandSolder, F.Cu at (152.3, 38.6)
- added R21: 0 RS, Resistor_SMD:R_0603_1608Metric_Pad0.98x0.95mm_HandSolder, F.Cu at (152.3, 41.1)
- added R22: 0 RS, Resistor_SMD:R_0603_1608Metric_Pad0.98x0.95mm_HandSolder, F.Cu at (152.3, 43.6)
- added R23: 0 C, Resistor_SMD:R_0603_1608Metric_Pad0.98x0.95mm_HandSolder, F.Cu at (152.3, 46.1)
- added R24: 0 C, Resistor_SMD:R_0603_1608Metric_Pad0.98x0.95mm_HandSolder, F.Cu at (152.3, 48.6)
- added R25: 0 RS, Resistor_SMD:R_0603_1608Metric_Pad0.98x0.95mm_HandSolder, F.Cu at (152.3, 51.1)
- added R26: 0 RS, Resistor_SMD:R_0603_1608Metric_Pad0.98x0.95mm_HandSolder, F.Cu at (152.3, 53.6)
- added R27: 120, Resistor_SMD:R_0805_2012Metric_Pad1.20x1.40mm_HandSolder, F.Cu at (166.0, 33.8)
- added R28: 0 RS, Resistor_SMD:R_0603_1608Metric_Pad0.98x0.95mm_HandSolder, F.Cu at (152.3, 56.2)
- added R29: 0 RS, Resistor_SMD:R_0603_1608Metric_Pad0.98x0.95mm_HandSolder, F.Cu at (156.6, 33.6)
- added R3: 10K, Resistor_SMD:R_0805_2012Metric_Pad1.20x1.40mm_HandSolder, F.Cu at (141.0, 108.7)
- added R30: 10k , RS, Resistor_SMD:R_0805_2012Metric_Pad1.20x1.40mm_HandSolder, F.Cu at (166.0, 36.7)
- added R31: 10k , RS, Resistor_SMD:R_0805_2012Metric_Pad1.20x1.40mm_HandSolder, F.Cu at (166.0, 39.7)
- added R32: 10k , RS, Resistor_SMD:R_0805_2012Metric_Pad1.20x1.40mm_HandSolder, F.Cu at (166.0, 42.6)
- added R33: 10k , RS, Resistor_SMD:R_0805_2012Metric_Pad1.20x1.40mm_HandSolder, F.Cu at (166.0, 45.6)
- added R34: 120, Resistor_SMD:R_0805_2012Metric_Pad1.20x1.40mm_HandSolder, F.Cu at (166.0, 48.5)
- added R35: 120, Resistor_SMD:R_0805_2012Metric_Pad1.20x1.40mm_HandSolder, F.Cu at (166.0, 51.5)
- added R36: 0 C, Resistor_SMD:R_0603_1608Metric_Pad0.98x0.95mm_HandSolder, F.Cu at (156.6, 36.1)
- added R37: 0 C, Resistor_SMD:R_0603_1608Metric_Pad0.98x0.95mm_HandSolder, F.Cu at (156.6, 38.6)
- added R38: 0 C, Resistor_SMD:R_0603_1608Metric_Pad0.98x0.95mm_HandSolder, F.Cu at (156.6, 41.1)
- added R39: 0 C, Resistor_SMD:R_0603_1608Metric_Pad0.98x0.95mm_HandSolder, F.Cu at (156.6, 43.6)
- added R4: 10K, Resistor_SMD:R_0805_2012Metric_Pad1.20x1.40mm_HandSolder, F.Cu at (141.0, 111.6)
- added R40: 120, Resistor_SMD:R_0805_2012Metric_Pad1.20x1.40mm_HandSolder, F.Cu at (166.0, 54.4)
- added R41: 330, Resistor_SMD:R_0603_1608Metric_Pad0.98x0.95mm_HandSolder, F.Cu at (167.7, 119.7)
- added R42: 10k LDO, Resistor_SMD:R_0805_2012Metric_Pad1.20x1.40mm_HandSolder, F.Cu at (198.4, 110.1)
- added R43: 10k LDO, Resistor_SMD:R_0805_2012Metric_Pad1.20x1.40mm_HandSolder, F.Cu at (198.4, 113.1)
- added R44: 100k, Resistor_SMD:R_0805_2012Metric_Pad1.20x1.40mm_HandSolder, F.Cu at (198.4, 116.0)
- added R45: 100k, Resistor_SMD:R_0805_2012Metric_Pad1.20x1.40mm_HandSolder, F.Cu at (198.4, 119.0)
- added R46: 24.9k, Resistor_SMD:R_0805_2012Metric_Pad1.20x1.40mm_HandSolder, F.Cu at (198.4, 121.9)
- added R47: 59, Resistor_SMD:R_0603_1608Metric_Pad0.98x0.95mm_HandSolder, F.Cu at (156.6, 46.1)
- added R48: 59, Resistor_SMD:R_0603_1608Metric_Pad0.98x0.95mm_HandSolder, F.Cu at (156.6, 48.6)
- added R5: 1k, Resistor_SMD:R_0805_2012Metric_Pad1.20x1.40mm_HandSolder, F.Cu at (141.0, 114.6)
- added R6: 1k, Resistor_SMD:R_0805_2012Metric_Pad1.20x1.40mm_HandSolder, F.Cu at (141.0, 117.5)
- added R7: 330, Resistor_SMD:R_0603_1608Metric_Pad0.98x0.95mm_HandSolder, F.Cu at (154.5, 115.1)
- added R8: 330, Resistor_SMD:R_0603_1608Metric_Pad0.98x0.95mm_HandSolder, F.Cu at (154.5, 117.6)
- added R9: 10k, Resistor_SMD:R_0805_2012Metric_Pad1.20x1.40mm_HandSolder, F.Cu at (141.0, 120.5)
- added SW1: SW_Push, Button_Switch_SMD:SW_SPST_CK_RS282G05A3, F.Cu at (158.1, 121.5)
- added TP1: TestPoint, TestPoint:TestPoint_Pad_D2.5mm, F.Cu at (167.8, 85.4)
- added TP10: TestPoint, TestPoint:TestPoint_Pad_D2.5mm, F.Cu at (172.3, 103.6)
- added TP11: TestPoint, TestPoint:TestPoint_Pad_D2.5mm, F.Cu at (176.9, 85.4)
- added TP12: TestPoint, TestPoint:TestPoint_Pad_D2.5mm, F.Cu at (176.9, 89.9)
- added TP13: TestPoint, TestPoint:TestPoint_Pad_D2.5mm, F.Cu at (176.9, 94.5)
- added TP14: TestPoint, TestPoint:TestPoint_Pad_D2.5mm, F.Cu at (176.9, 99.0)
- added TP15: TestPoint, TestPoint:TestPoint_Pad_D2.5mm, F.Cu at (122.6, 85.4)
- added TP16: TestPoint, TestPoint:TestPoint_Pad_D2.5mm, F.Cu at (122.6, 89.9)
- added TP17: TestPoint, TestPoint:TestPoint_Pad_D2.5mm, F.Cu at (122.6, 94.5)
- added TP18: TestPoint, TestPoint:TestPoint_Pad_D2.5mm, F.Cu at (122.6, 99.0)
- added TP19: TestPoint, TestPoint:TestPoint_Pad_D2.5mm, F.Cu at (127.2, 85.4)
- added TP2: TestPoint, TestPoint:TestPoint_Pad_D2.5mm, F.Cu at (167.8, 89.9)
- added TP20: TestPoint, TestPoint:TestPoint_Pad_D2.5mm, F.Cu at (127.2, 89.9)
- added TP21: TestPoint, TestPoint:TestPoint_Pad_D2.5mm, F.Cu at (127.2, 94.5)
- added TP22: TestPoint, TestPoint:TestPoint_Pad_D2.5mm, F.Cu at (127.2, 99.0)
- added TP23: TestPoint, TestPoint:TestPoint_Pad_D2.5mm, F.Cu at (131.7, 85.4)
- added TP24: TestPoint, TestPoint:TestPoint_Pad_D2.5mm, F.Cu at (131.7, 89.9)
- added TP25: TestPoint, TestPoint:TestPoint_Pad_D2.5mm, F.Cu at (131.7, 94.5)
- added TP26: TestPoint, TestPoint:TestPoint_Pad_D2.5mm, F.Cu at (131.7, 99.0)
- added TP27: TestPoint, TestPoint:TestPoint_Pad_D2.5mm, F.Cu at (136.3, 85.4)
- added TP28: TestPoint, TestPoint:TestPoint_Pad_D2.5mm, F.Cu at (136.3, 89.9)
- added TP29: TestPoint, TestPoint:TestPoint_Pad_D2.5mm, F.Cu at (136.3, 94.5)
- added TP3: TestPoint, TestPoint:TestPoint_Pad_D2.5mm, F.Cu at (167.8, 94.5)
- added TP30: TestPoint, TestPoint:TestPoint_Pad_D2.5mm, F.Cu at (136.3, 99.0)
- added TP31: TestPoint, TestPoint:TestPoint_Pad_D2.5mm, F.Cu at (140.8, 85.4)
- added TP32: TestPoint, TestPoint:TestPoint_Pad_D2.5mm, F.Cu at (140.8, 89.9)
- added TP33: TestPoint, TestPoint:TestPoint_Pad_D2.5mm, F.Cu at (140.8, 94.5)
- added TP34: TestPoint, TestPoint:TestPoint_Pad_D2.5mm, F.Cu at (140.8, 99.0)
- added TP35: TestPoint, TestPoint:TestPoint_Pad_D2.5mm, F.Cu at (113.4, 34.6)
- added TP36: TestPoint, TestPoint:TestPoint_Pad_D2.5mm, F.Cu at (113.4, 39.1)
- added TP37: TestPoint, TestPoint:TestPoint_Pad_D2.5mm, F.Cu at (113.4, 43.7)
- added TP38: TestPoint, TestPoint:TestPoint_Pad_D2.5mm, F.Cu at (113.4, 48.2)
- added TP39: TestPoint, TestPoint:TestPoint_Pad_D2.5mm, F.Cu at (113.4, 52.8)
- added TP4: TestPoint, TestPoint:TestPoint_Pad_D2.5mm, F.Cu at (167.8, 99.0)
- added TP40: TestPoint, TestPoint:TestPoint_Pad_D2.5mm, F.Cu at (113.4, 57.3)
- added TP41: TestPoint, TestPoint:TestPoint_Pad_D2.5mm, F.Cu at (113.4, 61.9)
- added TP42: TestPoint, TestPoint:TestPoint_Pad_D2.5mm, F.Cu at (118.0, 34.6)
- added TP43: TestPoint, TestPoint:TestPoint_Pad_D2.5mm, F.Cu at (118.0, 39.1)
- added TP44: TestPoint, TestPoint:TestPoint_Pad_D2.5mm, F.Cu at (118.0, 43.7)
- added TP45: TestPoint, TestPoint:TestPoint_Pad_D2.5mm, F.Cu at (118.0, 48.2)
- added TP46: TestPoint, TestPoint:TestPoint_Pad_D2.5mm, F.Cu at (118.0, 52.8)
- added TP47: TestPoint, TestPoint:TestPoint_Pad_D2.5mm, F.Cu at (118.0, 57.3)
- added TP48: TestPoint, TestPoint:TestPoint_Pad_D2.5mm, F.Cu at (118.0, 61.9)
- added TP49: TestPoint, TestPoint:TestPoint_Pad_D2.5mm, F.Cu at (122.5, 34.6)
- added TP5: TestPoint, TestPoint:TestPoint_Pad_D2.5mm, F.Cu at (167.8, 103.6)
- added TP50: TestPoint, TestPoint:TestPoint_Pad_D2.5mm, F.Cu at (122.5, 39.1)
- added TP51: TestPoint, TestPoint:TestPoint_Pad_D2.5mm, F.Cu at (122.5, 43.7)
- added TP52: TestPoint, TestPoint:TestPoint_Pad_D2.5mm, F.Cu at (122.5, 48.2)
- added TP53: TestPoint, TestPoint:TestPoint_Pad_D2.5mm, F.Cu at (122.5, 52.8)
- added TP54: TestPoint, TestPoint:TestPoint_Pad_D2.5mm, F.Cu at (122.5, 57.3)
- added TP55: TestPoint, TestPoint:TestPoint_Pad_D2.5mm, F.Cu at (122.5, 61.9)
- added TP56: TestPoint, TestPoint:TestPoint_Pad_D2.5mm, F.Cu at (127.1, 34.6)
- added TP57: TestPoint, TestPoint:TestPoint_Pad_D2.5mm, F.Cu at (127.1, 39.1)
- added TP58: TestPoint, TestPoint:TestPoint_Pad_D2.5mm, F.Cu at (127.1, 43.7)
- added TP59: TestPoint, TestPoint:TestPoint_Pad_D2.5mm, F.Cu at (127.1, 48.2)
- added TP6: TestPoint, TestPoint:TestPoint_Pad_D2.5mm, F.Cu at (172.3, 85.4)
- added TP60: TestPoint, TestPoint:TestPoint_Pad_D2.5mm, F.Cu at (127.1, 52.8)
- added TP61: TestPoint, TestPoint:TestPoint_Pad_D2.5mm, F.Cu at (127.1, 57.3)
- added TP62: TestPoint, TestPoint:TestPoint_Pad_D2.5mm, F.Cu at (127.1, 61.9)
- added TP7: TestPoint, TestPoint:TestPoint_Pad_D2.5mm, F.Cu at (172.3, 89.9)
- added TP8: TestPoint, TestPoint:TestPoint_Pad_D2.5mm, F.Cu at (172.3, 94.5)
- added TP9: TestPoint, TestPoint:TestPoint_Pad_D2.5mm, F.Cu at (172.3, 99.0)
- added U1: STM32F446RETx, Package_QFP:LQFP-64_10x10mm_P0.5mm, F.Cu at (150.3, 90.3)
- added U2: ISO1042BQDWVRQ1, ISO1042BQDWVRQ1:IC_AMC1311BQDWVQ1, F.Cu at (260.4, 90.2)
- added U3: ISO3082DW, Package_SO:SOIC-16W_7.5x10.3mm_P1.27mm, F.Cu at (245.1, 110.5)
- added U4: ISO3082DW, Package_SO:SOIC-16W_7.5x10.3mm_P1.27mm, F.Cu at (243.8, 97.8)
- added U5: ISO1042BQDWVRQ1, ISO1042BQDWVRQ1:IC_AMC1311BQDWVQ1, F.Cu at (260.4, 99.1)
- added U6: CRE1S0505S3C, Converter_DCDC:Converter_DCDC_Murata_CRE1xxxxxx3C_THT, F.Cu at (255.9, 45.8)
- added U7: CRE1S0505S3C, Converter_DCDC:Converter_DCDC_Murata_CRE1xxxxxx3C_THT, F.Cu at (259.8, 109.3)
- added U8: LP3963-3.3, Package_TO_SOT_SMD:TO-263-5_TabPin3, F.Cu at (189.9, 89.3)
- added Y1: 8_MHz, ECS-2520MVLC_8MHz:ECS2520MVLC080BNTR, F.Cu at (160.5, 98.0)
- added Y2: 32.768_KHz, Crystal:Crystal_SMD_MicroCrystal_CC8V-T1A-2Pin_2.0x1.2mm, F.Cu at (122.5, 130.8)
Other:
- copper layers 0 -> 4
