File: Design/Rapid_Core-RCP.kicad_pcb (KiCad board)
At the start: 4 copper layers, 145 x 70 mm, 154 parts, among them IC1 TLIN1039DDFRQ1, IC2 TLIN1039DDFRQ1, IC3 SHT30A-DIS-B2.5KS, IC4 LM60440ARPKR, J1 LIN-2, J10 RS-485-1, J11 RS-485-2, J12 CAN-2, J13 Input Power, J2 LIN-1, J3 LIN-1, J4 LIN-2, J5 GPIO_CONN_X_4, J6 SWD_Debug, J7 SPI, J8 USART, J9 CAN-1, SW1 SW_Push, U1 STM32F446RETx, U2 ISO1042BQDWVRQ1, U3 ISO3082DW, U4 ISO3082DW, U5 ISO1042BQDWVRQ1, U6 LP3963-3.3, U7 CRE1S0505S3C, U8 CRE1S0505S3C, Y1 Crystal_GND24, Y2 32.768_KHz

Commit message: Added Information to all the sheets
Parts:
- removed D8: SM712_SOT23, Package_TO_SOT_SMD:SOT-23
- removed J1: LIN-2, Connector_PinHeader_2.54mm:PinHeader_1x02_P2.54mm_Vertical
- added C49: 10uF, 10V, 0805, Capacitor_SMD:C_0805_2012Metric_Pad1.18x1.45mm_HandSolder, F.Cu at (163.4, 57.3)
- added C50: 0u1F, 10V, 0603, Capacitor_SMD:C_0603_1608Metric_Pad1.08x0.95mm_HandSolder, F.Cu at (177.9, 57.7)
- added C63: 4700pF, Capacitor_SMD:C_0805_2012Metric_Pad1.18x1.45mm_HandSolder, F.Cu at (236.8, 56.0)
- added C64: 10uf, Capacitor_SMD:C_0805_2012Metric_Pad1.18x1.45mm_HandSolder, F.Cu at (236.8, 59.0)
- added D10: GREEN, LED_SMD:LED_0603_1608Metric_Pad1.05x0.95mm_HandSolder, F.Cu at (76.2, 123.0)
- added G1: Not_to_bin, Not_To_Bin:Not_To_Bin, F.Cu at (42.4, 93.1)
- added J14: XT60PW-F, XT60PW-F_Connector:AMASS_XT60PW-F, F.Cu at (55.8, 49.2)
- added Q1: NMOS, Package_TO_SOT_SMD:SuperSOT-3, F.Cu at (76.5, 109.5)
- added Q2: NMOS, Package_TO_SOT_SMD:SuperSOT-3, F.Cu at (76.5, 114.3)
- added R43: 59, Resistor_SMD:R_0603_1608Metric_Pad0.98x0.95mm_HandSolder, F.Cu at (286.5, 61.8)
- added R44: 100 1% 1/5W, Resistor_SMD:R_0603_1608Metric_Pad0.98x0.95mm_HandSolder, F.Cu at (71.8, 108.2)
- added R45: 100 1% 1/5W, Resistor_SMD:R_0603_1608Metric_Pad0.98x0.95mm_HandSolder, F.Cu at (71.8, 110.7)
- added R46: 100 1% 1/5W, Resistor_SMD:R_0603_1608Metric_Pad0.98x0.95mm_HandSolder, F.Cu at (71.8, 113.2)
- added R47: 150, Resistor_SMD:R_0603_1608Metric_Pad0.98x0.95mm_HandSolder, F.Cu at (71.8, 115.7)
- added R48: 150, Resistor_SMD:R_0603_1608Metric_Pad0.98x0.95mm_HandSolder, F.Cu at (71.8, 118.2)
- added R49: 100k 1% 1/5W, Resistor_SMD:R_0603_1608Metric_Pad0.98x0.95mm_HandSolder, F.Cu at (71.8, 120.7)
- added R50: 100k 1% 1/5W, Resistor_SMD:R_0603_1608Metric_Pad0.98x0.95mm_HandSolder, F.Cu at (71.8, 123.2)
- added TP1: TestPoint, TestPoint:TestPoint_Pad_D1.0mm, F.Cu at (86.6, 60.3)
- added TP10: TestPoint, TestPoint:TestPoint_Pad_D1.0mm, F.Cu at (225.9, 96.4)
- added TP11: TestPoint, TestPoint:TestPoint_Pad_D1.0mm, F.Cu at (225.9, 99.5)
- added TP12: TestPoint, TestPoint:TestPoint_Pad_D1.0mm, F.Cu at (241.2, 84.2)
- added TP13: TestPoint, TestPoint:TestPoint_Pad_D1.0mm, F.Cu at (241.2, 87.2)
- added TP14: TestPoint, TestPoint:TestPoint_Pad_D1.0mm, F.Cu at (181.4, 48.3)
- added TP15: TestPoint, TestPoint:TestPoint_Pad_D1.0mm, F.Cu at (181.4, 51.3)
- added TP16: TestPoint, TestPoint:TestPoint_Pad_D1.0mm, F.Cu at (240.8, 53.0)
- added TP17: TestPoint, TestPoint:TestPoint_Pad_D1.0mm, F.Cu at (240.8, 56.1)
- added TP18: TestPoint, TestPoint:TestPoint_Pad_D1.0mm, F.Cu at (240.8, 59.1)
- added TP19: TestPoint, TestPoint:TestPoint_Pad_D1.0mm, F.Cu at (240.8, 62.2)
- added TP2: TestPoint, TestPoint:TestPoint_Pad_D1.0mm, F.Cu at (86.6, 63.4)
- added TP20: TestPoint, TestPoint:TestPoint_Pad_D1.0mm, F.Cu at (271.1, 52.0)
- added TP21: TestPoint, TestPoint:TestPoint_Pad_D1.0mm, F.Cu at (243.8, 53.0)
- added TP22: TestPoint, TestPoint:TestPoint_Pad_D1.0mm, F.Cu at (243.8, 56.1)
- added TP23: TestPoint, TestPoint:TestPoint_Pad_D1.0mm, F.Cu at (243.8, 59.1)
- added TP24: TestPoint, TestPoint:TestPoint_Pad_D1.0mm, F.Cu at (243.8, 62.2)
- added TP25: TestPoint, TestPoint:TestPoint_Pad_D1.0mm, F.Cu at (274.1, 52.0)
- added TP3: TestPoint, TestPoint:TestPoint_Pad_D1.0mm, F.Cu at (86.6, 66.4)
- added TP4: TestPoint, TestPoint:TestPoint_Pad_D1.0mm, F.Cu at (135.7, 86.4)
- added TP5: TestPoint, TestPoint:TestPoint_Pad_D1.0mm, F.Cu at (135.7, 89.5)
- added TP6: TestPoint, TestPoint:TestPoint_Pad_D1.0mm, F.Cu at (219.8, 96.4)
- added TP7: TestPoint, TestPoint:TestPoint_Pad_D1.0mm, F.Cu at (219.8, 99.5)
- added TP8: TestPoint, TestPoint:TestPoint_Pad_D1.0mm, F.Cu at (222.9, 96.4)
- added TP9: TestPoint, TestPoint:TestPoint_Pad_D1.0mm, F.Cu at (222.9, 99.5)
- C1: value 10uF -> 66uF LDO; footprint Capacitor_SMD:C_0805_2012Metric_Pad1.18x1.45mm_HandSolder -> Capacitor_SMD:CP_Elec_5x5.8
- C10: value 0u1F -> 100uF 1mohm; footprint Capacitor_SMD:C_0603_1608Metric_Pad1.08x0.95mm_HandSolder -> Capacitor_SMD:C_0805_2012Metric_Pad1.18x1.45mm_HandSolder
- C11: value 15pf -> 100uF 1mohm; footprint Capacitor_SMD:C_0603_1608Metric -> Capacitor_SMD:C_0805_2012Metric_Pad1.18x1.45mm_HandSolder
- C12: value 15pF -> 100uF, 30mohm,; footprint Capacitor_SMD:C_0603_1608Metric -> Capacitor_SMD:C_0805_2012Metric_Pad1.18x1.45mm_HandSolder
- C13: value 0u1F -> 20pF, 0603; footprint Capacitor_SMD:C_0603_1608Metric_Pad1.08x0.95mm_HandSolder -> Capacitor_SMD:C_0603_1608Metric
- C14: value 10uf -> 20pF; footprint Capacitor_SMD:C_0805_2012Metric_Pad1.18x1.45mm_HandSolder -> Capacitor_SMD:C_0603_1608Metric
- C15: value 1uf -> 15pf; footprint Capacitor_SMD:C_0603_1608Metric_Pad1.08x0.95mm_HandSolder -> Capacitor_SMD:C_0603_1608Metric
- C16: value 0.1uf -> 15pF; footprint Capacitor_SMD:C_0603_1608Metric_Pad1.08x0.95mm_HandSolder -> Capacitor_SMD:C_0603_1608Metric
- C17: value 4.7uf 6.3V XR7 -> 10uf
- C18, C37, C38: value 0.1uf -> 10uf; footprint Capacitor_SMD:C_0603_1608Metric_Pad1.08x0.95mm_HandSolder -> Capacitor_SMD:C_0805_2012Metric_Pad1.18x1.45mm_HandSolder
- C19: value 10uf -> 1uf; footprint Capacitor_SMD:C_0805_2012Metric_Pad1.18x1.45mm_HandSolder -> Capacitor_SMD:C_0603_1608Metric_Pad1.08x0.95mm_HandSolder
- C2: value 0u1F -> 4u7F 1mOhm; footprint Capacitor_SMD:C_0603_1608Metric_Pad1.08x0.95mm_HandSolder -> Capacitor_SMD:C_0805_2012Metric_Pad1.18x1.45mm_HandSolder
- C20, C26: value 1uf -> 0.1uf
- C21: value 0.1uf -> 1uf
- C25, C34, C42, C43: value 10uf -> 0.1uf; footprint Capacitor_SMD:C_0805_2012Metric_Pad1.18x1.45mm_HandSolder -> Capacitor_SMD:C_0603_1608Metric_Pad1.08x0.95mm_HandSolder
- C27: value 0.1uf -> 4.7uf 6.3V XR7; footprint Capacitor_SMD:C_0603_1608Metric_Pad1.08x0.95mm_HandSolder -> Capacitor_SMD:C_0805_2012Metric_Pad1.18x1.45mm_HandSolder
- C28: value 0.1uf -> 10uF; footprint Capacitor_SMD:C_0603_1608Metric_Pad1.08x0.95mm_HandSolder -> Capacitor_SMD:C_0805_2012Metric_Pad1.18x1.45mm_HandSolder
- C29: value 1uf -> 0.1uF
- C3, C4: value 220uF -> 0.22uF 1m; footprint Capacitor_SMD:C_0805_2012Metric_Pad1.18x1.45mm_HandSolder -> Capacitor_SMD:C_0603_1608Metric_Pad1.08x0.95mm_HandSolder
- C30: value 0.1uf -> 0u1F
- C41: value 10uf -> 4700pF
- C44: value 1uf -> 4700pF; footprint Capacitor_SMD:C_0603_1608Metric_Pad1.08x0.95mm_HandSolder -> Capacitor_SMD:C_0805_2012Metric_Pad1.18x1.45mm_HandSolder
- C45: value 0.1uf -> 220uF, 0805; footprint Capacitor_SMD:C_0603_1608Metric_Pad1.08x0.95mm_HandSolder -> Capacitor_SMD:C_0805_2012Metric_Pad1.18x1.45mm_HandSolder
- C46: value 10uf -> 220uF, 0805
- C47: value 1uf -> 10uF, 10V, 0805; footprint Capacitor_SMD:C_0603_1608Metric_Pad1.08x0.95mm_HandSolder -> Capacitor_SMD:C_0805_2012Metric_Pad1.18x1.45mm_HandSolder
- C48: value 0.1uf -> 0u1F, 10V, 0603
- C5: value 20pF -> 1uF 6.065m; footprint Capacitor_SMD:C_0603_1608Metric -> Capacitor_SMD:C_0603_1608Metric_Pad1.08x0.95mm_HandSolder
- C51: value 4u7F 1mOhm -> 0.1uf; footprint Capacitor_SMD:C_0805_2012Metric_Pad1.18x1.45mm_HandSolder -> Capacitor_SMD:C_0603_1608Metric_Pad1.08x0.95mm_HandSolder
- C52: value 0.22uF 1m -> 0.1uf
- C53: value 66uF LDO -> 1uf; footprint Capacitor_SMD:CP_Elec_5x5.8 -> Capacitor_SMD:C_0603_1608Metric_Pad1.08x0.95mm_HandSolder
- C54: value 0.22uF 1m -> 1uf
- C55, C56: value 1uF 6.065m -> 10uf; footprint Capacitor_SMD:C_0603_1608Metric_Pad1.08x0.95mm_HandSolder -> Capacitor_SMD:C_0805_2012Metric_Pad1.18x1.45mm_HandSolder
- C57: value 33uF LDO -> 0.1uf; footprint Capacitor_SMD:CP_Elec_4x5.8 -> Capacitor_SMD:C_0603_1608Metric_Pad1.08x0.95mm_HandSolder
- C58: value 0.1uF 1m -> 0.1uf
- C59: value 27pF 1mohm -> 1uf; footprint Capacitor_SMD:C_0805_2012Metric_Pad1.18x1.45mm_HandSolder -> Capacitor_SMD:C_0603_1608Metric_Pad1.08x0.95mm_HandSolder
- C6: value 20pF -> 33uF LDO; footprint Capacitor_SMD:C_0603_1608Metric -> Capacitor_SMD:CP_Elec_4x5.8
- C60: value 100uF 1mohm -> 4700pF
- C61: value 100uF 1mohm -> 1uf; footprint Capacitor_SMD:C_0805_2012Metric_Pad1.18x1.45mm_HandSolder -> Capacitor_SMD:C_0603_1608Metric_Pad1.08x0.95mm_HandSolder
- C62: value 100uF 30mohm -> 10uf
- C7: value 10uF -> 1uF 6.065m; footprint Capacitor_SMD:C_0805_2012Metric_Pad1.18x1.45mm_HandSolder -> Capacitor_SMD:C_0603_1608Metric_Pad1.08x0.95mm_HandSolder
- C8: value 0u1F -> 0.1uF 1m
- C9: value 10uF -> 27pF 1mohm
- D1, D2: value D -> SM712_SOT23; footprint Diode_SMD:D_SOD-323_HandSoldering -> Package_TO_SOT_SMD:SOT-23
- D3, D4: value RED -> D; footprint LED_SMD:LED_0603_1608Metric_Pad1.05x0.95mm_HandSolder -> Diode_SMD:D_SOD-323_HandSoldering
- D7: value SM712_SOT23 -> RED; footprint Package_TO_SOT_SMD:SOT-23 -> LED_SMD:LED_0603_1608Metric_Pad1.05x0.95mm_HandSolder
- D9: value RED -> GREEN
- G2: value Not_to_bin -> NOON_REAY_ENERGIES; footprint Not_To_Bin:Not_To_Bin -> Noon_Ray:Noon_Ray
- G3: value NOON_REAY_ENERGIES -> High_Voltage_Warning; footprint Noon_Ray:Noon_Ray -> High_Voltage_Warning_logo:High_Voltage_Warning
- G4: value High_Voltage_Warning -> ESD_Protection; footprint High_Voltage_Warning_logo:High_Voltage_Warning -> ESD_Protection_Sign:ESD_Protection_Sign
- IC1: value TLIN1039DDFRQ1 -> LM60440ARPKR; footprint TLIN1039DDFRQ1:SOT65P280X110-8N -> LM60440ARPKR_Buck:LM60440AQRPKRQ1
- IC2: value TLIN1039DDFRQ1 -> SHT30A-DIS-B2.5KS; footprint TLIN1039DDFRQ1:SOT65P280X110-8N -> SHT30A-DIS-B2.5KS:SON50P250X250X100-9N-D
- IC3: value SHT30A-DIS-B2.5KS -> TLIN1039DDFRQ1; footprint SHT30A-DIS-B2.5KS:SON50P250X250X100-9N-D -> TLIN1039DDFRQ1:SOT65P280X110-8N
- IC4: value LM60440ARPKR -> TLIN1039DDFRQ1; footprint LM60440ARPKR_Buck:LM60440AQRPKRQ1 -> TLIN1039DDFRQ1:SOT65P280X110-8N
- J10: value RS-485-1 -> LIN-1
- J11: value RS-485-2 -> LIN-2
- J12: value CAN-2 -> RS-485-1
- J13: value Input Power -> RS-485-2; footprint TerminalBlock_Phoenix:TerminalBlock_Phoenix_MKDS-1,5-2_1x02_P5.00mm_Horizontal -> 0530480210_2pin_P1.25_PicoBlade:MOLEX_530480210
- J2: value LIN-1 -> GPIO_CONN_X_4; footprint Connector_PinHeader_2.54mm:PinHeader_1x02_P2.54mm_Vertical -> Connector_PinHeader_2.54mm:PinHeader_1x06_P2.54mm_Vertical
- J3: value LIN-1 -> SPI; footprint 0530480210_2pin_P1.25_PicoBlade:MOLEX_530480210 -> Connector_PinHeader_2.54mm:PinHeader_1x05_P2.54mm_Vertical
- J4: value LIN-2 -> USART; footprint 0530480210_2pin_P1.25_PicoBlade:MOLEX_530480210 -> Connector_PinHeader_2.54mm:PinHeader_1x04_P2.54mm_Vertical
- J5: value GPIO_CONN_X_4 -> SWD_Debug; footprint Connector_PinHeader_2.54mm:PinHeader_1x06_P2.54mm_Vertical -> Connector_PinHeader_2.54mm:PinHeader_1x05_P2.54mm_Vertical
- J6: value SWD_Debug -> CAN-2; footprint Connector_PinHeader_2.54mm:PinHeader_1x05_P2.54mm_Vertical -> 0530480210_2pin_P1.25_PicoBlade:MOLEX_530480210
- J7: value SPI -> CAN-1; footprint Connector_PinHeader_2.54mm:PinHeader_1x05_P2.54mm_Vertical -> 0530480210_2pin_P1.25_PicoBlade:MOLEX_530480210
- J8: value USART -> LIN-2; footprint Connector_PinHeader_2.54mm:PinHeader_1x04_P2.54mm_Vertical -> Connector_PinHeader_2.54mm:PinHeader_1x02_P2.54mm_Vertical
- J9: value CAN-1 -> LIN-1; footprint 0530480210_2pin_P1.25_PicoBlade:MOLEX_530480210 -> Connector_PinHeader_2.54mm:PinHeader_1x02_P2.54mm_Vertical
- L1: value ACT45B-510-2P-TL003 -> 8.2mH 24mohm; footprint ACT45B-510-2P-TL003:IND_ACT45R_TDK -> Inductor_SMD:L_Coilcraft_XAL6060-XXX
- L5: value 8.2 24mohm -> ACT45B-510-2P-TL003; footprint Inductor_SMD:L_Coilcraft_XAL6060-XXX -> ACT45B-510-2P-TL003:IND_ACT45R_TDK
- R1, R2: value 10K -> 10k LDO
- R10: value 10k -> 0 C
- R13, R14, R15, R16, R17: value 0 RS -> 0 C
- R18, R21: value 0 RS -> 59; footprint Resistor_SMD:R_0805_2012Metric_Pad1.20x1.40mm_HandSolder -> Resistor_SMD:R_0603_1608Metric_Pad0.98x0.95mm_HandSolder
- R19, R20: value 0 C -> 59; footprint Resistor_SMD:R_0805_2012Metric_Pad1.20x1.40mm_HandSolder -> Resistor_SMD:R_0603_1608Metric_Pad0.98x0.95mm_HandSolder
- R22: value 0 RS -> 10K
- R23: value 120 -> 10K; footprint Resistor_SMD:R_2512_6332Metric_Pad1.40x3.35mm_HandSolder -> Resistor_SMD:R_0805_2012Metric_Pad1.20x1.40mm_HandSolder
- R24, R25: value 0 RS -> 1k
- R26, R27, R28, R29: value 10k , RS -> 0 RS
- R3, R4: value 4k7 -> 100k
- R30, R31: value 120 -> 0 RS; footprint Resistor_SMD:R_2512_6332Metric_Pad1.40x3.35mm_HandSolder -> Resistor_SMD:R_0805_2012Metric_Pad1.20x1.40mm_HandSolder
- R32, R33, R34, R35: value 0 C -> 0 RS
- R36: value 120 -> 10k , RS; footprint Resistor_SMD:R_2512_6332Metric_Pad1.40x3.35mm_HandSolder -> Resistor_SMD:R_0805_2012Metric_Pad1.20x1.40mm_HandSolder
- R37, R39: value 10k LDO -> 10k , RS
- R38: value 330 -> 10k , RS; footprint Resistor_SMD:R_0603_1608Metric_Pad0.98x0.95mm_HandSolder -> Resistor_SMD:R_0805_2012Metric_Pad1.20x1.40mm_HandSolder
- R40, R41: value 100k -> 59; footprint Resistor_SMD:R_0805_2012Metric_Pad1.20x1.40mm_HandSolder -> Resistor_SMD:R_0603_1608Metric_Pad0.98x0.95mm_HandSolder
- R42: value 24.9k -> 59; footprint Resistor_SMD:R_0805_2012Metric_Pad1.20x1.40mm_HandSolder -> Resistor_SMD:R_0603_1608Metric_Pad0.98x0.95mm_HandSolder
- R5: value 1k -> 24.9k
- R6: value 1k -> 10k
- R7, R8: value 330 -> 4k7; footprint Resistor_SMD:R_0603_1608Metric_Pad0.98x0.95mm_HandSolder -> Resistor_SMD:R_0805_2012Metric_Pad1.20x1.40mm_HandSolder
- U1: value STM32F446RETx -> LP3963-3.3; footprint Package_QFP:LQFP-64_10x10mm_P0.5mm -> Package_TO_SOT_SMD:TO-263-5_TabPin3
- U2: value ISO1042BQDWVRQ1 -> CRE1S0505S3C; footprint ISO1042BQDWVRQ1:IC_AMC1311BQDWVQ1 -> Converter_DCDC:Converter_DCDC_Murata_CRE1xxxxxx3C_THT
- U3: value ISO3082DW -> CRE1S0505S3C; footprint Package_SO:SOIC-16W_7.5x10.3mm_P1.27mm -> Converter_DCDC:Converter_DCDC_Murata_CRE1xxxxxx3C_THT
- U4: value ISO3082DW -> STM32F446RETx; footprint Package_SO:SOIC-16W_7.5x10.3mm_P1.27mm -> Package_QFP:LQFP-64_10x10mm_P0.5mm
- U6: value LP3963-3.3 -> ISO1042BQDWVRQ1; footprint Package_TO_SOT_SMD:TO-263-5_TabPin3 -> ISO1042BQDWVRQ1:IC_AMC1311BQDWVQ1
- U7, U8: value CRE1S0505S3C -> ISO3082DW; footprint Converter_DCDC:Converter_DCDC_Murata_CRE1xxxxxx3C_THT -> Package_SO:SOIC-16W_7.5x10.3mm_P1.27mm
- Y1: value Crystal_GND24 -> 32.768_KHz; footprint Crystal:Crystal_SMD_2520-4Pin_2.5x2.0mm -> Crystal:Crystal_SMD_MicroCrystal_CC8V-T1A-2Pin_2.0x1.2mm
- Y2: value 32.768_KHz -> Crystal_GND24; footprint Crystal:Crystal_SMD_MicroCrystal_CC8V-T1A-2Pin_2.0x1.2mm -> Crystal:Crystal_SMD_2520-4Pin_2.5x2.0mm
- moved R42 194.1 mm to (286.5, 59.3), turned to 0 degrees
- moved R41 191.0 mm to (286.5, 56.8)
- moved R40 189.7 mm to (286.5, 54.3)
- moved R39 183.0 mm to (257.2, 61.9), turned to 0 degrees
- moved R37 180.9 mm to (257.2, 56.0), turned to 0 degrees
- moved J13 177.4 mm to (250.4, 45.3), turned to 0 degrees
- moved R38 172.9 mm to (257.2, 58.9)
- moved D2 169.8 mm to (272.4, 79.7), turned to 0 degrees
- moved D1 152.1 mm to (272.4, 75.1), turned to 0 degrees
- moved C55 151.8 mm to (236.8, 43.9)
- moved C56 150.5 mm to (236.8, 47.0)
- moved J7 150.0 mm to (264.2, 88.4), turned to 0 degrees
- moved C60 143.7 mm to (236.8, 50.0)
- moved C62 142.7 mm to (236.8, 53.0)
- moved C43 128.1 mm to (278.7, 78.1), turned to 0 degrees
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Connections:
- C1 pad 1: +3.3V -> +5V
- C11 pad 1: GND1 -> +5V
- C11 pad 2: /RCC_OSC_32_IN -> GND1
- C12 pad 1: GND1 -> +5V
- C12 pad 2: /RCC_OSC_32_OUT -> GND1
- C13 pad 1: /NRST -> GND1
- C13 pad 2: GND1 -> /Project_Architecture/MCU/HSE_IN
- C14 pad 1: +3.3V -> GND1
- C14 pad 2: GND1 -> /Project_Architecture/MCU/HSE_OUT
- C15 pad 1: +3.3V -> GND1
- C15 pad 2: GND1 -> /Project_Architecture/MCU/RCC_OSC_32_IN
- C16 pad 1: +3.3V -> GND1
- C16 pad 2: GND1 -> /Project_Architecture/MCU/RCC_OSC_32_OUT
- C17 pad 1: /VCAP -> +3.3V
- C2 pad 1: +3.3V -> +24V
- C27 pad 1: +3.3V -> /Project_Architecture/MCU/VCAP
- C28 pad 1: GND1 -> +3.3V
- C28 pad 2: +3.3V -> GND1
- C3 pad 1: /LIN1 -> +24V
- C30 pad 1: +3.3V -> /Project_Architecture/GPIO/NRST
- C31 pad 1: GND1 -> +3.3V
- C31 pad 2: +3.3V -> GND1
- C33 pad 1: GND1 -> +3.3V
- C33 pad 2: +3.3V -> GND1
- C34 pad 1: +5VA -> GND1
- C34 pad 2: GND2 -> +3.3V
- C35 pad 1: +5VA -> +3.3V
- C35 pad 2: GND2 -> GND1
- C36 pad 1: +5VA -> GND1
- C36 pad 2: GND2 -> +3.3V
- C38 pad 1: GND2 -> +5VA
- C38 pad 2: +5VA -> GND2
- C4 pad 1: /LIN2 -> +24V
- C41 pad 1: GND2 -> /Project_Architecture/Comm - Isolated_CAN/CAN_2_Cap
- C41 pad 2: +5VA -> GND2
- C43 pad 1: +3.3V -> GND2
- C43 pad 2: GND1 -> +5VA
- C44 pad 1: +3.3V -> /Project_Architecture/Comm - Isolated_CAN/CAN_2_Cap
- C44 pad 2: GND1 -> GND2
- C45 pad 1: GND1 -> /Project_Architecture/Comm - LIN/LIN1
- C45 pad 2: +3.3V -> GND1
- C46 pad 1: +5VA -> /Project_Architecture/Comm - LIN/LIN2
- C46 pad 2: GND2 -> GND1
- C47 pad 1: +5VA -> +5V
- C47 pad 2: GND2 -> GND1
- C48 pad 1: GND2 -> +5V
- C48 pad 2: +5VA -> GND1
- C5 pad 1: GND1 -> /Project_Architecture/Power - Generation/LM_VCC
- C5 pad 2: /HSE_IN -> GND1
- C51 pad 1: +24V -> +3.3V
- C52 pad 1: +24V -> +3.3V
- C53 pad 1: +5V -> +3.3V
- C54 pad 1: +24V -> +3.3V
- C55 pad 1: /Power_Stage/LM_VCC -> GND1
- C55 pad 2: GND1 -> +3.3V
- C56 pad 1: /Power_Stage/LM_VCC -> GND1
- C56 pad 2: GND1 -> +3.3V
- C57 pad 1: +3.3V -> +5VA
- C57 pad 2: GND1 -> GND2
- C58 pad 1: /Power_Stage/LM_BOOT -> +5VA
- C58 pad 2: /Power_Stage/LM_SW -> GND2
- C59 pad 1: +5V -> +5VA
- C59 pad 2: /Power_Stage/LM_FB -> GND2
- C6 pad 1: GND1 -> +3.3V
- C6 pad 2: /HSE_OUT -> GND1
- C60 pad 1: +5V -> /Project_Architecture/Comm - Isolated_RS-485/RS-485_1_Cap
- C60 pad 2: GND1 -> GND2
- C61 pad 1: +5V -> +5VA
- C61 pad 2: GND1 -> GND2
- C62 pad 1: +5V -> GND2
- C62 pad 2: GND1 -> +5VA
- C7 pad 1: +5V -> /Project_Architecture/Power - Generation/LM_VCC
- C8 pad 1: +5V -> /Project_Architecture/Power - Generation/LM_BOOT
- C8 pad 2: GND1 -> /Project_Architecture/Power - Generation/LM_SW
- C9 pad 2: GND1 -> /Project_Architecture/Power - Generation/LM_FB
- D1 pad 1: /LIN1_CMD -> /Project_Architecture/Comm - Isolated_CAN/CAN_H_IN-2
- D1 pad 2: +5V -> /Project_Architecture/Comm - Isolated_CAN/CAN_L_IN-2
- D2 pad 1: /LIN2_CMD -> /Project_Architecture/Comm - Isolated_CAN/CAN_H_IN-1
- D2 pad 2: +5V -> /Project_Architecture/Comm - Isolated_CAN/CAN_L_IN-1
- D3 pad 1: /LED_1 -> /Project_Architecture/Comm - LIN/LIN2_CMD
- D3 pad 2: +3.3V -> +5V
- D4 pad 1: /LED_2 -> /Project_Architecture/Comm - LIN/LIN1_CMD
- D4 pad 2: +3.3V -> +5V
- D5 pad 1: /Communication_interface/CAN_H_IN-1 -> /Project_Architecture/Comm - Isolated_RS-485/RS-485_B_IN-1
- D5 pad 2: /Communication_interface/CAN_L_IN-1 -> /Project_Architecture/Comm - Isolated_RS-485/RS-485_A-IN-1
- D6 pad 1: /Communication_interface/RS-485_B_IN-1 -> /Project_Architecture/Comm - Isolated_RS-485/RS-485_B_IN-2
- D6 pad 2: /Communication_interface/RS-485_A-IN-1 -> /Project_Architecture/Comm - Isolated_RS-485/RS-485_A_IN-2
- D7 pad 1: /Communication_interface/RS-485_B_IN-2 -> GND1
- D7 pad 2: /Communication_interface/RS-485_A_IN-2 -> /Project_Architecture/Indication - USR/PWR_LED
- D9 pad 1: /Power_Stage/PWR_LED -> /Project_Architecture/Indication - USR/LED_1_D
- D9 pad 2: +3.3V -> /Project_Architecture/Indication - USR/LED_1_R
- IC1 pad 1: /LIN1_RX -> GND1
- IC1 pad 2: /LIN1_EN -> +24V
- IC1 pad 3: unconnected-(IC1-NC_1-Pad3) -> /Project_Architecture/Power - Generation/LM_SW
- IC1 pad 4: /LIN1_TX -> /Project_Architecture/Power - Generation/LM_BOOT
- IC1 pad 5: GND1 -> /Project_Architecture/Power - Generation/LM_VCC
- IC1 pad 6: /LIN1 -> GND1
- IC1 pad 7: +5V -> /Project_Architecture/Power - Generation/LM_FB
- IC1 pad 8: unconnected-(IC1-NC_2-Pad8) -> /Project_Architecture/Power - Generation/LM_PG
- IC2 pad 1: /LIN2_RX -> /Project_Architecture/MCU/I2C_SDA_HUM
- IC2 pad 2: /LIN2_EN -> GND1
- IC2 pad 4: /LIN2_TX -> /Project_Architecture/MCU/I2C_SCL_HUM
- IC2 pad 5: GND1 -> +3.3V
- IC2 pad 6: /LIN2 -> unconnected-(IC2-NRESET-Pad6)
- IC2 pad 7: +5V -> GND1
- IC2 pad 8: unconnected-(IC2-NC_2-Pad8) -> GND1
- IC3 pad 1: /I2C_SDA_HUM -> /Project_Architecture/Comm - LIN/LIN1_RX
- IC3 pad 2: GND1 -> /Project_Architecture/Comm - LIN/LIN1_EN
- IC3 pad 4: /I2C_SCL_HUM -> /Project_Architecture/Comm - LIN/LIN1_TX
- IC3 pad 5: +3.3V -> GND1
- IC3 pad 6: unconnected-(IC3-NRESET-Pad6) -> /Project_Architecture/Comm - LIN/LIN1
- IC3 pad 7: GND1 -> +5V
- IC3 pad 8: GND1 -> unconnected-(IC3-NC_2-Pad8)
- IC4 pad 1: GND1 -> /Project_Architecture/Comm - LIN/LIN2_RX
- IC4 pad 2: +24V -> /Project_Architecture/Comm - LIN/LIN2_EN
- IC4 pad 3: /Power_Stage/LM_SW -> unconnected-(IC4-NC_1-Pad3)
- IC4 pad 4: /Power_Stage/LM_BOOT -> /Project_Architecture/Comm - LIN/LIN2_TX
- IC4 pad 5: /Power_Stage/LM_VCC -> GND1
- IC4 pad 6: GND1 -> /Project_Architecture/Comm - LIN/LIN2
- IC4 pad 7: /Power_Stage/LM_FB -> +5V
- IC4 pad 8: /Power_Stage/LM_PG -> unconnected-(IC4-NC_2-Pad8)
- J10 pad 1: /Communication_interface/RS-485_A-IN-1 -> GND1
- J10 pad 2: /Communication_interface/RS-485_B_IN-1 -> /Project_Architecture/Comm - LIN/LIN1
- J11 pad 1: /Communication_interface/RS-485_A_IN-2 -> GND1
- J11 pad 2: /Communication_interface/RS-485_B_IN-2 -> /Project_Architecture/Comm - LIN/LIN2
- J12 pad 1: /Communication_interface/CAN_L_IN-2 -> /Project_Architecture/Comm - Isolated_RS-485/RS-485_A-IN-1
- J12 pad 2: /Communication_interface/CAN_H_IN-2 -> /Project_Architecture/Comm - Isolated_RS-485/RS-485_B_IN-1
- J13 pad 1: +24V -> /Project_Architecture/Comm - Isolated_RS-485/RS-485_A_IN-2
- J13 pad 2: GND1 -> /Project_Architecture/Comm - Isolated_RS-485/RS-485_B_IN-2
- J2 pad 1: /LIN1_CMD_R -> +3.3V
- J2 pad 2: /LIN1 -> /Project_Architecture/GPIO/GPIO_1_PB0
- J3 pad 1: GND1 -> +3.3V
- J3 pad 2: /LIN1 -> /Project_Architecture/GPIO/SPI1_SCK
- J4 pad 1: GND1 -> +3.3V
- J4 pad 2: /LIN2 -> /Project_Architecture/GPIO/USART2_TX
- J5 pad 2: /GPIO_1_PB0 -> /Project_Architecture/GPIO/SW_CLK
- J5 pad 3: /GPIO_1_PB1 -> /Project_Architecture/GPIO/NRST
- J5 pad 4: /GPIO_1_PB2 -> /Project_Architecture/GPIO/SWDIO
- J5 pad 5: /GPIO_1_PB3 -> GND1
- J6 pad 1: +3.3V -> /Project_Architecture/Comm - Isolated_CAN/CAN_L_IN-2
- J6 pad 2: /SW_CLK -> /Project_Architecture/Comm - Isolated_CAN/CAN_H_IN-2
- J7 pad 1: +3.3V -> /Project_Architecture/Comm - Isolated_CAN/CAN_L_IN-1
- J7 pad 2: /SPI1_SCK -> /Project_Architecture/Comm - Isolated_CAN/CAN_H_IN-1
- J8 pad 1: +3.3V -> /Project_Architecture/Comm - LIN/LIN2_CMD_R
- J8 pad 2: /USART2_TX -> /Project_Architecture/Comm - LIN/LIN2
- J9 pad 1: /Communication_interface/CAN_L_IN-1 -> /Project_Architecture/Comm - LIN/LIN1_CMD_R
- J9 pad 2: /Communication_interface/CAN_H_IN-1 -> /Project_Architecture/Comm - LIN/LIN1
- L1 pad 1: /Communication_interface/CAN_H-1 -> /Project_Architecture/Power - Generation/LM_SW
- L1 pad 2: /Communication_interface/CAN_L-1 -> +5V
- L2 pad 1: /Communication_interface/RS-485_B-1 -> /Project_Architecture/Comm - Isolated_CAN/CAN_H-2
- L2 pad 2: /Communication_interface/RS-485_A-1 -> /Project_Architecture/Comm - Isolated_CAN/CAN_L-2
- L2 pad 3: /Communication_interface/RS-485_A-IN-1 -> /Project_Architecture/Comm - Isolated_CAN/CAN_L_IN-2
- L2 pad 4: /Communication_interface/RS-485_B_IN-1 -> /Project_Architecture/Comm - Isolated_CAN/CAN_H_IN-2
- L3 pad 1: /Communication_interface/RS-485_B-2 -> /Project_Architecture/Comm - Isolated_CAN/CAN_H-1
- L3 pad 2: /Communication_interface/RS-485_A-2 -> /Project_Architecture/Comm - Isolated_CAN/CAN_L-1
- L3 pad 3: /Communication_interface/RS-485_A_IN-2 -> /Project_Architecture/Comm - Isolated_CAN/CAN_L_IN-1
- L3 pad 4: /Communication_interface/RS-485_B_IN-2 -> /Project_Architecture/Comm - Isolated_CAN/CAN_H_IN-1
- L4 pad 1: /Communication_interface/CAN_H-2 -> /Project_Architecture/Comm - Isolated_RS-485/RS-485_B-1
- L4 pad 2: /Communication_interface/CAN_L-2 -> /Project_Architecture/Comm - Isolated_RS-485/RS-485_A-1
- L4 pad 3: /Communication_interface/CAN_L_IN-2 -> /Project_Architecture/Comm - Isolated_RS-485/RS-485_A-IN-1
- L4 pad 4: /Communication_interface/CAN_H_IN-2 -> /Project_Architecture/Comm - Isolated_RS-485/RS-485_B_IN-1
- L5 pad 1: /Power_Stage/LM_SW -> /Project_Architecture/Comm - Isolated_RS-485/RS-485_B-2
- L5 pad 2: +5V -> /Project_Architecture/Comm - Isolated_RS-485/RS-485_A-2
- R1 pad 2: /LIN1_RX -> /Project_Architecture/Power - Generation/LDO_SH
- R10 pad 1: /BOOT0 -> /Project_Architecture/Comm - Isolated_CAN/CAN2_TX
- R10 pad 2: GND1 -> /Project_Architecture/Comm - Isolated_CAN/CAN2_TX_R-2
- R11 pad 1: CAN1_TX -> /Project_Architecture/Comm - Isolated_CAN/CAN2_RX
- R11 pad 2: /Communication_interface/CAN1_TX_R-1 -> /Project_Architecture/Comm - Isolated_CAN/CAN2_RX_R-2
- R12 pad 1: CAN1_RX -> /Project_Architecture/Comm - Isolated_CAN/CAN1_TX
- R12 pad 2: /Communication_interface/CAN1_RX_R-1 -> /Project_Architecture/Comm - Isolated_CAN/CAN1_TX_R-1
- R13 pad 1: RS-485_1_TX -> /Project_Architecture/Comm - Isolated_CAN/CAN1_RX
- R13 pad 2: /Communication_interface/RS-485_1_TX_R-1 -> /Project_Architecture/Comm - Isolated_CAN/CAN1_RX_R-1
- R14 pad 1: RS-485_1_RX -> /Project_Architecture/Comm - Isolated_CAN/CAN_H-2
- R14 pad 2: /Communication_interface/RS-485_1_RX_R-1 -> /Project_Architecture/Comm - Isolated_CAN/CAN_H_IN-2
- R15 pad 1: RS-485_1_EN -> /Project_Architecture/Comm - Isolated_CAN/CAN_L-2
- R15 pad 2: /Communication_interface/RS-485_1_EN_R-1 -> /Project_Architecture/Comm - Isolated_CAN/CAN_L_IN-2
- R16 pad 1: RS-485_2_TX -> /Project_Architecture/Comm - Isolated_CAN/CAN_H-1
- R16 pad 2: /Communication_interface/RS-485_2_TX_R-2 -> /Project_Architecture/Comm - Isolated_CAN/CAN_H_IN-1
- R17 pad 1: RS-485_2_RX -> /Project_Architecture/Comm - Isolated_CAN/CAN_L-1
- R17 pad 2: /Communication_interface/RS-485_2_RX_R-2 -> /Project_Architecture/Comm - Isolated_CAN/CAN_L_IN-1
- R18 pad 1: RS-485_2_EN -> /Project_Architecture/Comm - Isolated_CAN/CAN_H_IN-2
- R18 pad 2: /Communication_interface/RS-485_2_EN_R-2 -> /Project_Architecture/Comm - Isolated_CAN/CAN_2_Cap
- R19 pad 1: /Communication_interface/CAN_H-1 -> /Project_Architecture/Comm - Isolated_CAN/CAN_2_Cap
- R19 pad 2: /Communication_interface/CAN_H_IN-1 -> /Project_Architecture/Comm - Isolated_CAN/CAN_L_IN-2
- R2 pad 1: +5V -> /Project_Architecture/Power - Generation/LDO_ERR
- R2 pad 2: /LIN2_RX -> +3.3V
- R20 pad 1: /Communication_interface/CAN_L-1 -> /Project_Architecture/Comm - Isolated_CAN/CAN_H_IN-1
- R20 pad 2: /Communication_interface/CAN_L_IN-1 -> /Project_Architecture/Comm - Isolated_CAN/CAN_2_Cap
- R21 pad 1: /Communication_interface/RS-485_B-1 -> /Project_Architecture/Comm - Isolated_CAN/CAN_2_Cap
- R21 pad 2: /Communication_interface/RS-485_B_IN-1 -> /Project_Architecture/Comm - Isolated_CAN/CAN_L_IN-1
- R22 pad 1: /Communication_interface/RS-485_A-1 -> +5V
- R22 pad 2: /Communication_interface/RS-485_A-IN-1 -> /Project_Architecture/Comm - LIN/LIN2_RX
- R23 pad 1: /Communication_interface/CAN_H_IN-1 -> +5V
- R23 pad 2: /Communication_interface/CAN_L_IN-1 -> /Project_Architecture/Comm - LIN/LIN1_RX
- R24 pad 1: /Communication_interface/RS-485_A-2 -> /Project_Architecture/Comm - LIN/LIN2_CMD_R
- R24 pad 2: /Communication_interface/RS-485_A_IN-2 -> /Project_Architecture/Comm - LIN/LIN2_CMD
- R25 pad 1: /Communication_interface/RS-485_B-2 -> /Project_Architecture/Comm - LIN/LIN1_CMD_R
- R25 pad 2: /Communication_interface/RS-485_B_IN-2 -> /Project_Architecture/Comm - LIN/LIN1_CMD
- R26 pad 1: /Communication_interface/RS-485_B-2 -> /Project_Architecture/Comm - Isolated_RS-485/RS-485_1_TX
- R26 pad 2: GND2 -> /Project_Architecture/Comm - Isolated_RS-485/RS-485_1_TX_R-1
- R27 pad 1: /Communication_interface/RS-485_A-2 -> /Project_Architecture/Comm - Isolated_RS-485/RS-485_1_RX
- R27 pad 2: +5VA -> /Project_Architecture/Comm - Isolated_RS-485/RS-485_1_RX_R-1
- R28 pad 1: /Communication_interface/RS-485_B-1 -> /Project_Architecture/Comm - Isolated_RS-485/RS-485_1_EN
- R28 pad 2: GND2 -> /Project_Architecture/Comm - Isolated_RS-485/RS-485_1_EN_R-1
- R29 pad 1: /Communication_interface/RS-485_A-1 -> /Project_Architecture/Comm - Isolated_RS-485/RS-485_2_TX
- R29 pad 2: +5VA -> /Project_Architecture/Comm - Isolated_RS-485/RS-485_2_TX_R-2
- R3 pad 1: +3.3V -> /Project_Architecture/Power - Generation/LM_PG
- R3 pad 2: /I2C_SDA_HUM -> +5V
- R30 pad 1: /Communication_interface/RS-485_B_IN-1 -> /Project_Architecture/Comm - Isolated_RS-485/RS-485_2_RX
- R30 pad 2: /Communication_interface/RS-485_A-IN-1 -> /Project_Architecture/Comm - Isolated_RS-485/RS-485_2_RX_R-2
- R31 pad 1: /Communication_interface/RS-485_B_IN-2 -> /Project_Architecture/Comm - Isolated_RS-485/RS-485_2_EN
- R31 pad 2: /Communication_interface/RS-485_A_IN-2 -> /Project_Architecture/Comm - Isolated_RS-485/RS-485_2_EN_R-2
- R32 pad 1: CAN2_TX -> /Project_Architecture/Comm - Isolated_RS-485/RS-485_B-1
- R32 pad 2: /Communication_interface/CAN2_TX_R-2 -> /Project_Architecture/Comm - Isolated_RS-485/RS-485_B_IN-1
- R33 pad 1: CAN2_RX -> /Project_Architecture/Comm - Isolated_RS-485/RS-485_A-1
- R33 pad 2: /Communication_interface/CAN2_RX_R-2 -> /Project_Architecture/Comm - Isolated_RS-485/RS-485_A-IN-1
- R34 pad 1: /Communication_interface/CAN_H-2 -> /Project_Architecture/Comm - Isolated_RS-485/RS-485_A-2
- R34 pad 2: /Communication_interface/CAN_H_IN-2 -> /Project_Architecture/Comm - Isolated_RS-485/RS-485_A_IN-2
- R35 pad 1: /Communication_interface/CAN_L-2 -> /Project_Architecture/Comm - Isolated_RS-485/RS-485_B-2
- R35 pad 2: /Communication_interface/CAN_L_IN-2 -> /Project_Architecture/Comm - Isolated_RS-485/RS-485_B_IN-2
- R36 pad 1: /Communication_interface/CAN_H_IN-2 -> /Project_Architecture/Comm - Isolated_RS-485/RS-485_B-2
- R36 pad 2: /Communication_interface/CAN_L_IN-2 -> GND2
- R37 pad 1: +5V -> /Project_Architecture/Comm - Isolated_RS-485/RS-485_A-2
- R37 pad 2: /Power_Stage/LDO_SH -> +5VA
- R38 pad 1: /Power_Stage/PWR_LED -> /Project_Architecture/Comm - Isolated_RS-485/RS-485_B-1
- R38 pad 2: GND1 -> GND2
- R39 pad 1: /Power_Stage/LDO_ERR -> /Project_Architecture/Comm - Isolated_RS-485/RS-485_A-1
- R39 pad 2: +3.3V -> +5VA
- R4 pad 1: +3.3V -> /Project_Architecture/Power - Generation/LM_FB
- R4 pad 2: /I2C_SCL_HUM -> +5V
- R40 pad 1: /Power_Stage/LM_PG -> /Project_Architecture/Comm - Isolated_RS-485/RS-485_B_IN-1
- R40 pad 2: +5V -> /Project_Architecture/Comm - Isolated_RS-485/RS-485_1_Cap
- R41 pad 1: /Power_Stage/LM_FB -> /Project_Architecture/Comm - Isolated_RS-485/RS-485_1_Cap
- R41 pad 2: +5V -> /Project_Architecture/Comm - Isolated_RS-485/RS-485_A-IN-1
- R42 pad 1: GND1 -> /Project_Architecture/Comm - Isolated_RS-485/RS-485_B_IN-2
- R42 pad 2: /Power_Stage/LM_FB -> /Project_Architecture/Comm - Isolated_RS-485/RS-485_2_Cap
- R5 pad 1: /LIN2_CMD_R -> GND1
- R5 pad 2: /LIN2_CMD -> /Project_Architecture/Power - Generation/LM_FB
- R6 pad 1: /LIN1_CMD_R -> /Project_Architecture/MCU/BOOT0
- R6 pad 2: /LIN1_CMD -> GND1
- R7 pad 1: /LED_1 -> +3.3V
- R7 pad 2: /USR_LED_1 -> /Project_Architecture/MCU/I2C_SDA_HUM
- R8 pad 1: /LED_2 -> +3.3V
- R8 pad 2: /USR_LED_2 -> /Project_Architecture/MCU/I2C_SCL_HUM
- R9 pad 1: /NRST -> /Project_Architecture/GPIO/NRST
- SW1 pad 1: /NRST -> /Project_Architecture/GPIO/NRST
- U1 pad 1: +3.3V -> /Project_Architecture/Power - Generation/LDO_SH
- U1 pad 2: unconnected-(U1-PC13-Pad2) -> +5V
- U1 pad 3: /RCC_OSC_32_IN -> GND1
- U1 pad 4: /RCC_OSC_32_OUT -> +3.3V
- U1 pad 5: /HSE_IN -> /Project_Architecture/Power - Generation/LDO_ERR
- U2 pad 1: +3.3V -> GND1
- U2 pad 2: /Communication_interface/CAN1_TX_R-1 -> +5V
- U2 pad 3: /Communication_interface/CAN1_RX_R-1 -> GND2
- U2 pad 4: GND1 -> +5VA
- U3 pad 1: +3.3V -> GND1
- U3 pad 2: GND1 -> +5V
- U3 pad 3: /Communication_interface/RS-485_1_RX_R-1 -> GND2
- U3 pad 4: /Communication_interface/RS-485_1_EN_R-1 -> +5VA
- U4 pad 10: GND2 -> unconnected-(U4-PC2-Pad10)
- U4 pad 12: /Communication_interface/RS-485_A-2 -> GND1
- U4 pad 13: /Communication_interface/RS-485_B-2 -> +3.3V
- U4 pad 15: GND2 -> unconnected-(U4-PA1-Pad15)
- U4 pad 16: +5VA -> /Project_Architecture/GPIO/USART2_TX
- U4 pad 2: GND1 -> unconnected-(U4-PC13-Pad2)
- U4 pad 3: /Communication_interface/RS-485_2_RX_R-2 -> /Project_Architecture/MCU/RCC_OSC_32_IN
- U4 pad 4: /Communication_interface/RS-485_2_EN_R-2 -> /Project_Architecture/MCU/RCC_OSC_32_OUT
- U4 pad 5: /Communication_interface/RS-485_2_EN_R-2 -> /Project_Architecture/MCU/HSE_IN
- U4 pad 6: /Communication_interface/RS-485_2_TX_R-2 -> /Project_Architecture/MCU/HSE_OUT
- U4 pad 7: GND1 -> /Project_Architecture/GPIO/NRST
- U4 pad 8: GND1 -> unconnected-(U4-PC0-Pad8)
- U4 pad 9: GND2 -> unconnected-(U4-PC1-Pad9)
- U5 pad 2: /Communication_interface/CAN2_TX_R-2 -> /Project_Architecture/Comm - Isolated_CAN/CAN2_TX_R-2
- U5 pad 3: /Communication_interface/CAN2_RX_R-2 -> /Project_Architecture/Comm - Isolated_CAN/CAN2_RX_R-2
- U5 pad 6: /Communication_interface/CAN_L-2 -> /Project_Architecture/Comm - Isolated_CAN/CAN_L-2
- U5 pad 7: /Communication_interface/CAN_H-2 -> /Project_Architecture/Comm - Isolated_CAN/CAN_H-2
- U6 pad 1: /Power_Stage/LDO_SH -> +3.3V
- U6 pad 2: +5V -> /Project_Architecture/Comm - Isolated_CAN/CAN1_TX_R-1
- U6 pad 3: GND1 -> /Project_Architecture/Comm - Isolated_CAN/CAN1_RX_R-1
- U6 pad 4: +3.3V -> GND1
- U6 pad 5: /Power_Stage/LDO_ERR -> GND2
- U7 pad 1: GND1 -> +3.3V
- U7 pad 2: +5V -> GND1
- U7 pad 3: GND2 -> /Project_Architecture/Comm - Isolated_RS-485/RS-485_1_RX_R-1
- U7 pad 4: +5VA -> /Project_Architecture/Comm - Isolated_RS-485/RS-485_1_EN_R-1
- U8 pad 1: GND1 -> +3.3V
- U8 pad 2: +5V -> GND1
- U8 pad 3: GND2 -> /Project_Architecture/Comm - Isolated_RS-485/RS-485_2_RX_R-2
- U8 pad 4: +5VA -> /Project_Architecture/Comm - Isolated_RS-485/RS-485_2_EN_R-2
- Y1 pad 1: /HSE_OUT -> /Project_Architecture/MCU/RCC_OSC_32_OUT
- Y1 pad 2: GND1 -> /Project_Architecture/MCU/RCC_OSC_32_IN
- Y2 pad 1: /RCC_OSC_32_OUT -> /Project_Architecture/MCU/HSE_OUT
- Y2 pad 2: /RCC_OSC_32_IN -> GND1
Routing:
- net GND1: track 124.6 -> 0.00 mm, vias 101 -> 0
- net /NRST: track 67.9 -> 0.00 mm, vias 2 -> 0
- net GND2: track 63.8 -> 0.00 mm, vias 24 -> 0
- net /GPIO_1_PB3: track 41.9 -> 0.00 mm, vias 1 -> 0
- net CAN1_TX: track 38.4 -> 0.00 mm
- net CAN1_RX: track 38.1 -> 0.00 mm
- net /USR_LED_1: track 36.7 -> 0.00 mm, vias 2 -> 0
- net /SWDIO: track 35.7 -> 0.00 mm
- net +3.3V: track 35.1 -> 0.00 mm, vias 38 -> 0
- net /USR_LED_2: track 35.1 -> 0.00 mm, vias 2 -> 0
- net /LIN2_RX: track 30.0 -> 0.00 mm
- net CAN2_RX: track 29.3 -> 0.00 mm
- net /SW_CLK: track 28.8 -> 0.00 mm
- net CAN2_TX: track 27.8 -> 0.00 mm
- net /USART2_TX: track 27.6 -> 0.00 mm
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- removed copper zone on B.Cu, net +24V
- removed copper zone on F.Cu, net +24V
- removed copper zone on B.Cu, net +3.3V
- removed copper zone on F.Cu, net +3.3V
- removed copper zone on F.Cu, net +5V
- removed copper zone on B.Cu, net +5VA
- removed copper zone on F.Cu, net +5VA
- removed copper zone on F.Cu, net /Power_Stage/LM_FB
- removed copper zone on F.Cu, net /Power_Stage/LM_VCC
- removed copper zone on F.Cu, net GND1
- removed copper zone on In1.Cu, net GND1
- removed copper zone on In2.Cu, net GND1
- removed copper zone on In1.Cu, net GND2
- removed copper zone on In2.Cu, net GND2
Other:
- board outline removed
- board text removed: "+"
- board text removed: "3.3V"
- board text removed: "A"
- board text removed: "B"
- board text removed: "CAN-1"
- board text removed: "CAN-2"
- board text removed: "CAN-H"
- board text removed: "CAN-L"
- board text removed: "CLK"
- board text removed: "DIO"
- board text removed: "GND"
- board text removed: "GPIO"
- board text removed: "J10"
- board text removed: "J11"
- board text removed: "J12"
- board text removed: "J3"
- board text removed: "J4"
- board text removed: "J9"
- board text removed: "LIN"
- board text removed: "MISO"
- board text removed: "MOSI"
- board text removed: "NRST"
- board text removed: "NRST_SW"
- board text removed: "PB0"
- board text removed: "PB1"
- board text removed: "PB2"
- board text removed: "PB3"
- board text removed: "PWR_LED"
- board text removed: "RS-485-1"
- board text removed: "RS-485-2"
- board text removed: "RX"
- board text removed: "SCK"
- board text removed: "SPI"
- board text removed: "SWD"
- board text removed: "TX"
- board text removed: "U2"
- board text removed: "U5"
- board text removed: "UART"
- board text removed: "USR_1"
- board text removed: "USR_2"
