File: Design/Power_stage.kicad_sch (KiCad schematic)
At the start: 39 parts, among them IC4 LM60440ARPKR, J13 Input Power, U6 LP3963-3.3, U7 CRE1S0505S3C, U8 CRE1S0505S3C

Commit message: Added everything
Parts:
- added G2: Not_to_bin, Not_To_Bin:Not_To_Bin, symbol Not_To_Bin:Not_To_Bin
- added G3: NOON_REAY_ENERGIES, Noon_Ray:Noon_Ray, symbol Noon_Ray:Noon_Ray
- added G4: High_Voltage_Warning, High_Voltage_Warning_logo:High_Voltage_Warning, symbol High_Voltage_Warning:HIgh_Voltage_Warning
Other:
- note added: "Symbols"
Changed lines of the file:
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@@
 		(title "Rapid-Core")
 		(date "2024-09-09")
-		(rev "1.0.0")
+		(rev "1.0.1")
 	)
 	(junction
@@
 	)
 	(rectangle
+		(start 13.97 15.24)
+		(end 91.44 56.515)
+		(stroke
+			(width 0.5)
+			(type default)
+		)
+		(fill
+			(type none)
+		)
+	)
+	(rectangle
 		(start 298.45 24.13)
 		(end 298.45 24.13)
@@
 		)
 	)
+	(text "Symbols"
+		(exclude_from_sim no)
+		(at 19.05 17.272 0)
+		(effects
+			(font
+				(size 1.27 1.27)
+				(thickness 0.254)
+				(bold yes)
+			)
+		)
+	)
 	(text "LDO\n"
 		(exclude_from_sim no)
@@
 	)
 	(symbol
+		(lib_id "Not_To_Bin:Not_To_Bin")
+		(at 24.13 25.4 0)
+		(unit 1)
+		(exclude_from_sim no)
+		(in_bom yes)
+		(on_board yes)
+		(dnp no)
+		(property "Reference" "G2"
+			(at 22.86 21.59 0)
+			(effects
+				(font
+					(size 1.27 1.27)
+				)
+				(justify left)
+			)
+		)
+		(property "Value" "Not_to_bin"
+			(at 24.13 27.2675 0)
+			(effects
+				(font
+					(size 1.27 1.27)
+				)
+				(hide yes)
+			)
+		)
+		(property "Footprint" "Not_To_Bin:Not_To_Bin"
+			(at 24.13 25.4 0)
+			(effects
+				(font
+					(size 1.27 1.27)
+				)
+				(hide yes)
+			)
+		)
+		(property "Datasheet" ""
+			(at 24.13 25.4 0)
+			(effects
+				(font
+					(size 1.27 1.27)
+				)
+				(hide yes)
+			)
+		)
+		(property "Description" ""
+			(at 24.13 25.4 0)
+			(effects
+				(font
+					(size 1.27 1.27)
+				)
+				(hide yes)
+			)
+		)
+		(instances
+			(project ""
+				(path "/1a5d67a4-b410-4c7a-b64e-9e0193c8e6b4/03c0cb4f-19c3-413c-9319-70c93aa2053e"
+					(reference "G2")
+					(unit 1)
+				)
+			)
+		)
+	)
+	(symbol
 		(lib_name "GND1_1")
 		(lib_id "power:GND1")
@@
 	)
 	(symbol
+		(lib_id "High_Voltage_Warning:HIgh_Voltage_Warning")
+		(at 43.18 25.4 0)
+		(unit 1)
+		(exclude_from_sim no)
+		(in_bom yes)
+		(on_board yes)
+		(dnp no)
+		(fields_autoplaced yes)
+		(property "Reference" "G4"
+			(at 46.99 25.407 0)
+			(effects
+				(font
+					(size 1.27 1.27)
+				)
+				(justify left)
+			)
+		)
+		(property "Value" "High_Voltage_Warning"
+			(at 38.354 25.908 0)
+			(effects
+				(font
+					(size 1.27 1.27)
+				)
+				(hide yes)
+			)
+		)
+		(property "Footprint" "High_Voltage_Warning_logo:High_Voltage_Warning"
+			(at 43.434 30.48 0)
+			(effects
+				(font
+					(size 1.27 1.27)
+				)
+				(hide yes)
+			)
+		)
+		(property "Datasheet" ""
+			(at 43.18 25.4 0)
+			(effects
+				(font
+					(size 1.27 1.27)
+				)
+				(hide yes)
+			)
+		)
+		(property "Description" ""
+			(at 43.18 25.4 0)
+			(effects
+				(font
+					(size 1.27 1.27)
+				)
+				(hide yes)
+			)
+		)
+		(instances
+			(project ""
+				(path "/1a5d67a4-b410-4c7a-b64e-9e0193c8e6b4/03c0cb4f-19c3-413c-9319-70c93aa2053e"
+					(reference "G4")
+					(unit 1)
+				)
+			)
+		)
+	)
+	(symbol
 		(lib_id "Device:LED")
 		(at 110.49 128.27 180)
@@
 					(unit 1)
 				)
+			)
+		)
+	)
+	(symbol
+		(lib_id "Noon_Ray:Noon_Ray")
+		(at 31.75 25.4 0)
+		(unit 1)
+		(exclude_from_sim no)
+		(in_bom yes)
+		(on_board yes)
+		(dnp no)
+		(fields_autoplaced yes)
+		(property "Reference" "G3"
+			(at 36.83 25.4108 0)
+			(effects
+				(font
+					(size 1.27 1.27)
+				)
+				(justify left)
+			)
+		)
+		(property "Value" "NOON_REAY_ENERGIES"
+			(at 31.496 25.4 0)
+			(effects
+				(font
+					(size 1.27 1.27)
+				)
+				(hide yes)
+			)
+		)
+		(property "Footprint" "Noon_Ray:Noon_Ray"
+			(at 31.496 25.4 0)
+			(effects
+				(font
+					(size 1.27 1.27)
+				)
+				(hide yes)
+			)
+		)
+		(property "Datasheet" ""
+			(at 31.75 25.4 0)
+			(effects
+				(font
+					(size 1.27 1.27)
+				)
+				(hide yes)
+			)
+		)
+		(property "Description" ""
+			(at 31.75 25.4 0)
+			(effects
+				(font
+					(size 1.27 1.27)
+				)
+				(hide yes)
+			)
+		)
+		(instances
+			(project ""
+				(path "/1a5d67a4-b410-4c7a-b64e-9e0193c8e6b4/03c0cb4f-19c3-413c-9319-70c93aa2053e"
+					(reference "G3")
+					(unit 1)
+				)
