File: Design/Communication_interface.kicad_sch (KiCad schematic)
At the start: 87 parts, among them J10 RS-485-1, J11 RS-485-2, J12 CAN-2, J9 CAN-1, U2 ISO1042BQDWVRQ1, U3 ISO3082DW, U4 ISO3082DW, U5 ISO1042BQDWVRQ1

Commit message: Added Information to all the sheets
Parts:
- removed C27, C30, C36, C37: 0.1uf, Capacitor_SMD:C_0603_1608Metric_Pad1.08x0.95mm_HandSolder, symbol Device:C
- removed C29, C32, C39, C40: 1uf, Capacitor_SMD:C_0603_1608Metric_Pad1.08x0.95mm_HandSolder, symbol Device:C
- removed C31, C33, C41, C42: 10uf, Capacitor_SMD:C_0805_2012Metric_Pad1.18x1.45mm_HandSolder, symbol Device:C
- removed D6, D7: SM712_SOT23, Package_TO_SOT_SMD:SOT-23, symbol Diode:SM712_SOT23
- removed G1: High_Voltage_Warning, High_Voltage_Warning_logo:High_Voltage_Warning, symbol High_Voltage_Warning:HIgh_Voltage_Warning
- removed J10: RS-485-1, 0530480210_2pin_P1.25_PicoBlade:MOLEX_530480210, symbol 0530480210_2pin_P1.25_PicoBlade:530480210
- removed J11: RS-485-2, 0530480210_2pin_P1.25_PicoBlade:MOLEX_530480210, symbol 0530480210_2pin_P1.25_PicoBlade:530480210
- removed L2, L3: ACT45B-510-2P-TL003, ACT45B-510-2P-TL003:IND_ACT45R_TDK, symbol ACT45B-510-2P-TL003:ACT45B-510-2P-TL003
- removed R13, R14, R15, R16, R17, R18, R21, R22, R24, R25: 0 RS, Resistor_SMD:R_0805_2012Metric_Pad1.20x1.40mm_HandSolder, symbol Device:R
- removed R26, R27, R28, R29: 10k , RS, Resistor_SMD:R_0805_2012Metric_Pad1.20x1.40mm_HandSolder, symbol Device:R
- removed R30, R31: 120, Resistor_SMD:R_2512_6332Metric_Pad1.40x3.35mm_HandSolder, symbol Device:R
- removed TP20, TP21, TP22, TP23, TP24, TP25, TP28, TP29, TP30, TP31: TestPoint, TestPoint:TestPoint_Pad_D1.0mm, symbol Connector:TestPoint
- removed U3, U4: ISO3082DW, Package_SO:SOIC-16W_7.5x10.3mm_P1.27mm, symbol Interface_UART:ISO3082DW
Other:
- note removed: "RS-485 1"
- note removed: "RS-485 2"
