File: Design/Block_Diagram.kicad_sch (KiCad schematic)
At the start: 0 parts

Commit message: Project finished , man files generated
Other:
- note added: "[${#}] ${SHEETNAME}"
Changed lines of the file:
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@@
 		(rev "1.0.1")
 	)
+	(text "[${#}] ${SHEETNAME}"
+		(exclude_from_sim no)
+		(at 138.176 19.558 0)
+		(effects
+			(font
+				(face "Times New Roman")
+				(size 6 6)
+				(thickness 0.254)
+				(bold yes)
+				(color 159 72 15 1)
+			)
+		)
+	)
 )

Commit message: new Design for Prototyping
Other:
- title: Rapid-Core -> (none)
