File: Design/Comm - Isolated_CAN.kicad_sch (KiCad schematic)
At the start: 42 parts, among them J6 CAN-2, J7 CAN-1, U5 ISO1042BQDWVRQ1, U6 ISO1042BQDWVRQ1

Commit message: Layout complete
Parts:
- removed TP10, TP11, TP12, TP13, TP6, TP7, TP8, TP9: TestPoint, TestPoint:TestPoint_Pad_D1.0mm, symbol Connector:TestPoint
- added TP12, TP13, TP14, TP15, TP16, TP17, TP18, TP19: Test_point, Test_point:Test_point, symbol Test_point:Test_point
- C31: renamed from C33; value 10uf -> 10uF
- C32: renamed from C35; value 1uf -> 1uF
- C33: renamed from C36; value 0.1uf -> 0.1uF
- C34: renamed from C37; value 10uf -> 10uF
- C35: renamed from C39; value 1uf -> 1uF
- C36: renamed from C42; value 0.1uf -> 0.1uF
- C38: value 10uf -> 10uF
- C39: renamed from C40; value 1uf -> 1uF
- C40: renamed from C43; value 0.1uf -> 0.1uF
- C41: renamed from C31; value 10uf -> 10uF
- C42: renamed from C32; value 1uf -> 1uF
- C43: renamed from C34; value 0.1uf -> 0.1uF
- D2: renamed from D1; MANUFACTURER PART NO CDSOT23-SM712 -> (none)
- J6: renamed from J7; value CAN-1 -> CAN; MANUFACTURER Molex -> (none); MAXIMUM_PACKAGE_HEIGHT 3.5 mm -> (none); PARTREV A -> (none); STANDARD Manufacturer Recommendations -> (none); manufacturer Part No 0530480210 -> (none)
- J7: renamed from J6; value CAN-2 -> CAN; MANUFACTURER Molex -> (none); MANUFACTURER PART NO 0530480210 -> (none); MAXIMUM_PACKAGE_HEIGHT 3.5 mm -> (none); PARTREV A -> (none); STANDARD Manufacturer Recommendations -> (none)
- L2: renamed from L3; MANUFACTURER PART NO  744235510 -> (none)
- L3: renamed from L2; MANUFACTURER PART NO 744235510 -> (none)
- R10: renamed from R16; footprint Resistor_SMD:R_0805_2012Metric_Pad1.20x1.40mm_HandSolder -> Resistor_SMD:R_0402_1005Metric_Pad0.72x0.64mm_HandSolder
- R11: renamed from R20; footprint Resistor_SMD:R_0603_1608Metric_Pad0.98x0.95mm_HandSolder -> Resistor_SMD:R_0402_1005Metric_Pad0.72x0.64mm_HandSolder
- R12, R13: footprint Resistor_SMD:R_0805_2012Metric_Pad1.20x1.40mm_HandSolder -> Resistor_SMD:R_0402_1005Metric_Pad0.72x0.64mm_HandSolder
- R14: renamed from R21; footprint Resistor_SMD:R_0603_1608Metric_Pad0.98x0.95mm_HandSolder -> Resistor_SMD:R_0402_1005Metric_Pad0.72x0.64mm_HandSolder
- R15: renamed from R17; footprint Resistor_SMD:R_0805_2012Metric_Pad1.20x1.40mm_HandSolder -> Resistor_SMD:R_0402_1005Metric_Pad0.72x0.64mm_HandSolder
- R16: renamed from R14; footprint Resistor_SMD:R_0805_2012Metric_Pad1.20x1.40mm_HandSolder -> Resistor_SMD:R_0402_1005Metric_Pad0.72x0.64mm_HandSolder
- R17: renamed from R18; footprint Resistor_SMD:R_0603_1608Metric_Pad0.98x0.95mm_HandSolder -> Resistor_SMD:R_0402_1005Metric_Pad0.72x0.64mm_HandSolder
- R18: renamed from R10; footprint Resistor_SMD:R_0805_2012Metric_Pad1.20x1.40mm_HandSolder -> Resistor_SMD:R_0402_1005Metric_Pad0.72x0.64mm_HandSolder
- R19: renamed from R11; footprint Resistor_SMD:R_0805_2012Metric_Pad1.20x1.40mm_HandSolder -> Resistor_SMD:R_0402_1005Metric_Pad0.72x0.64mm_HandSolder
- R20: renamed from R19; footprint Resistor_SMD:R_0603_1608Metric_Pad0.98x0.95mm_HandSolder -> Resistor_SMD:R_0402_1005Metric_Pad0.72x0.64mm_HandSolder
- R21: renamed from R15; footprint Resistor_SMD:R_0805_2012Metric_Pad1.20x1.40mm_HandSolder -> Resistor_SMD:R_0402_1005Metric_Pad0.72x0.64mm_HandSolder
- renumbered C44 to C37, C41 to C44, D2 to D1, U6 to U5, U5 to U6
Connections:
- net CAN1_RX: now also TP13.1 (TP)
- net CAN1_TX: now also TP12.1 (TP)
- net CAN2_RX: now also TP17.1 (TP)
- net CAN2_TX: now also TP16.1 (TP)
- net CAN_2_Cap: no longer C37.1, R11.2, R14.1
- net CAN_H_IN-1: now also TP14.1 (TP)
- net CAN_H_IN-2: now also TP18.1 (TP)
- net CAN_L_IN-1: now also TP15.1 (TP)
- net CAN_L_IN-2: now also TP19.1 (TP)
- new net CAN_1_Cap: C37.1, R11.2, R14.1
Other:
- note added: "Test Points CAN - 1"
- note added: "Test Points CAN - 2"
- moved on the sheet: R12, R13

Commit message: new Design for Prototyping
Parts:
- removed J6, J7: CAN, 0530480210_2pin_P1.25_PicoBlade:MOLEX_530480210, symbol 0530480210_2pin_P1.25_PicoBlade:530480210
- removed TP14, TP15, TP18, TP19: Test_point, Test_point:Test_point, symbol Test_point:Test_point
- renumbered C31 to C34, C32 to C35, C33 to C36, C34 to C37, C35 to C38, C36 to C39, C37 to C40, C38 to C41, C39 to C42, C40 to C43, C41 to C44, C42 to C45, C43 to C46, C44 to C47, R12 to R10, R13 to R11, R14 to R12, R15 to R13, R16 to R14, R17 to R15, R18 to R16, R19 to R17, R20 to R18, R21 to R19, R10 to R8, R11 to R9, TP16 to TP11, TP17 to TP13, TP13 to TP14, U5 to U4, U6 to U5
Connections:
- net CAN_H_IN-1 renamed CAN_1_H
- net CAN_H_IN-2 renamed CAN_2_H
- net CAN_L_IN-1 renamed CAN_1_L
- net CAN_L_IN-2 renamed CAN_2_L
Other:
- title: Rapid-Core -> (none)
- moved on the sheet: C34, C35, C36, C37, C38, C39, C40, C41, C42, C43, C44, C45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
