File: Design/Comm - Isolated_RS-485.kicad_sch (KiCad schematic)
At the start: 50 parts, among them J12 RS-485-1, J13 RS-485-2, U7 ISO3082DW, U8 ISO3082DW

Commit message: Layout complete
Parts:
- removed TP16, TP17, TP18, TP19, TP20, TP21, TP22, TP23, TP24, TP25: TestPoint, TestPoint:TestPoint_Pad_D1.0mm, symbol Connector:TestPoint
- added TP28, TP29, TP30, TP31, TP32, TP33, TP34, TP35, TP36, TP37: Test_point, Test_point:Test_point, symbol Test_point:Test_point
- C51: renamed from C57; value 0.1uf -> 0.1uF
- C52: renamed from C59; value 1uf -> 1uF
- C53: renamed from C62; value 10uf -> 10uF
- C54: renamed from C51; value 0.1uf -> 0.1uF
- C55: renamed from C54; value 1uf -> 1uF
- C56: value 10uf -> 10uF
- C58: value 0.1uf -> 0.1uF
- C59: renamed from C61; value 1uf -> 1uF
- C60: renamed from C64; value 10uf -> 10uF
- C61: renamed from C52; value 0.1uf -> 0.1uF
- C62: renamed from C53; value 1uf -> 1uF
- C63: renamed from C55; value 10uf -> 10uF
- D5: MANUFACTURER PART NO  CDSOT23-SM712 -> (none)
- J12: value RS-485-1 -> RS-485; MANUFACTURER Molex -> (none); MANUFACTURER PART NO  0530480210 -> (none); MAXIMUM_PACKAGE_HEIGHT 3.5 mm -> (none); STANDARD Manufacturer Recommendations -> (none)
- J13: value RS-485-2 -> RS-485; MANUFACTURER Molex -> (none); MAXIMUM_PACKAGE_HEIGHT 3.5 mm -> (none); PARTREV A -> (none); STANDARD Manufacturer Recommendations -> (none)
- L4: MANUFACTURER PART NO  744235510 -> (none)
- L5: MANUFACTURER PART NO 744235510 -> (none)
- R26: renamed from R38; footprint Resistor_SMD:R_0805_2012Metric_Pad1.20x1.40mm_HandSolder -> Resistor_SMD:R_0603_1608Metric_Pad0.98x0.95mm_HandSolder
- R27: renamed from R32; footprint Resistor_SMD:R_0805_2012Metric_Pad1.20x1.40mm_HandSolder -> Resistor_SMD:R_0402_1005Metric_Pad0.72x0.64mm_HandSolder
- R28: renamed from R40; footprint Resistor_SMD:R_0603_1608Metric_Pad0.98x0.95mm_HandSolder -> Resistor_SMD:R_0402_1005Metric_Pad0.72x0.64mm_HandSolder
- R29: renamed from R26; footprint Resistor_SMD:R_0805_2012Metric_Pad1.20x1.40mm_HandSolder -> Resistor_SMD:R_0402_1005Metric_Pad0.72x0.64mm_HandSolder
- R30: renamed from R27; footprint Resistor_SMD:R_0805_2012Metric_Pad1.20x1.40mm_HandSolder -> Resistor_SMD:R_0402_1005Metric_Pad0.72x0.64mm_HandSolder
- R31: renamed from R41; footprint Resistor_SMD:R_0603_1608Metric_Pad0.98x0.95mm_HandSolder -> Resistor_SMD:R_0402_1005Metric_Pad0.72x0.64mm_HandSolder
- R32: renamed from R33; footprint Resistor_SMD:R_0805_2012Metric_Pad1.20x1.40mm_HandSolder -> Resistor_SMD:R_0402_1005Metric_Pad0.72x0.64mm_HandSolder
- R33: renamed from R28; value 0 RS -> 0 RS J
- R34: renamed from R39; footprint Resistor_SMD:R_0805_2012Metric_Pad1.20x1.40mm_HandSolder -> Resistor_SMD:R_0603_1608Metric_Pad0.98x0.95mm_HandSolder
- R35: renamed from R36; footprint Resistor_SMD:R_0805_2012Metric_Pad1.20x1.40mm_HandSolder -> Resistor_SMD:R_0603_1608Metric_Pad0.98x0.95mm_HandSolder
- R36: renamed from R35; footprint Resistor_SMD:R_0805_2012Metric_Pad1.20x1.40mm_HandSolder -> Resistor_SMD:R_0402_1005Metric_Pad0.72x0.64mm_HandSolder
- R37: renamed from R42; footprint Resistor_SMD:R_0603_1608Metric_Pad0.98x0.95mm_HandSolder -> Resistor_SMD:R_0402_1005Metric_Pad0.72x0.64mm_HandSolder
- R38: renamed from R29; footprint Resistor_SMD:R_0805_2012Metric_Pad1.20x1.40mm_HandSolder -> Resistor_SMD:R_0402_1005Metric_Pad0.72x0.64mm_HandSolder
- R39: renamed from R30; footprint Resistor_SMD:R_0805_2012Metric_Pad1.20x1.40mm_HandSolder -> Resistor_SMD:R_0402_1005Metric_Pad0.72x0.64mm_HandSolder
- R40: renamed from R43; footprint Resistor_SMD:R_0603_1608Metric_Pad0.98x0.95mm_HandSolder -> Resistor_SMD:R_0402_1005Metric_Pad0.72x0.64mm_HandSolder
- R41: renamed from R31; value 0 RS -> 0 RS J
- R42: renamed from R34; footprint Resistor_SMD:R_0805_2012Metric_Pad1.20x1.40mm_HandSolder -> Resistor_SMD:R_0402_1005Metric_Pad0.72x0.64mm_HandSolder
- R43: renamed from R37; footprint Resistor_SMD:R_0805_2012Metric_Pad1.20x1.40mm_HandSolder -> Resistor_SMD:R_0603_1608Metric_Pad0.98x0.95mm_HandSolder
- U7, U8: value ISO3082DW -> ISO3082DWR
- renumbered C60 to C57, C63 to C64
Connections:
- net RS-485_1_EN: now also TP30.1 (TP)
- net RS-485_1_RX: now also TP29.1 (TP)
- net RS-485_1_TX: now also TP28.1 (TP)
- net RS-485_2_EN: now also TP35.1 (TP)
- net RS-485_2_RX: now also TP34.1 (TP)
- net RS-485_2_TX: now also TP33.1 (TP)
- net RS-485_A-IN-1: now also TP32.1 (TP)
- net RS-485_A_IN-2: now also TP37.1 (TP)
- net RS-485_B_IN-1: now also TP31.1 (TP)
- net RS-485_B_IN-2: now also TP36.1 (TP)
Other:
- note added: "Test Points RS_485 - 1"
- note added: "Test Points RS_485 - 2"

Commit message: new Design for Prototyping
Parts:
- removed J12, J13: RS-485, 0530480210_2pin_P1.25_PicoBlade:MOLEX_530480210, symbol 0530480210_2pin_P1.25_PicoBlade:530480210
- removed TP31, TP32, TP36, TP37: Test_point, Test_point:Test_point, symbol Test_point:Test_point
- renumbered C51 to C54, C52 to C55, C53 to C56, C54 to C57, C55 to C58, C56 to C59, C57 to C60, C58 to C61, C59 to C62, C60 to C63, C61 to C64, C62 to C65, C63 to C66, C64 to C67, R26 to R24, R27 to R25, R28 to R26, R29 to R27, R30 to R28, R31 to R29, R32 to R30, R33 to R31, R34 to R32, R35 to R33, R36 to R34, R37 to R35, R38 to R36, R39 to R37, R40 to R38, R41 to R39, R42 to R40, R43 to R41, TP33 to TP23, TP28 to TP24, TP34 to TP25, TP29 to TP26, TP35 to TP27, TP30 to TP28, U7 to U6, U8 to U7
Connections:
- net RS-485_A-IN-1 renamed RS_485_1_A
- net RS-485_A_IN-2 renamed RS_485_2_A
- net RS-485_B_IN-1 renamed RS_485_1_B
- net RS-485_B_IN-2 renamed RS_485_2_B
Other:
- note removed: "RS-485 2"
- title: Rapid-Core -> (none)
- moved on the sheet: C54, C55, C56, C57, C58, C59, C60, C61, C62, C63, C64, C65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
