File: Design/Comm - LIN.kicad_sch (KiCad schematic)
At the start: 20 parts, among them IC3 TLIN1039DDFRQ1, IC4 TLIN1039DDFRQ1, J10 LIN-1, J11 LIN-2, J8 LIN-2, J9 LIN-1

Commit message: Layout complete
Parts:
- removed TP14, TP15: TestPoint, TestPoint:TestPoint_Pad_D1.0mm, symbol Connector:TestPoint
- added TP20, TP21, TP22, TP23, TP24, TP25, TP26, TP27: Test_point, Test_point:Test_point, symbol Test_point:Test_point
- C45: renamed from C47; value 10uF, 10V, 0805 -> 10uF
- C46: renamed from C48; value 0u1F, 10V, 0603 -> 0.1uF
- C47: renamed from C45; footprint Capacitor_SMD:C_0805_2012Metric_Pad1.18x1.45mm_HandSolder -> Capacitor_SMD:C_1206_3216Metric_Pad1.33x1.80mm_HandSolder
- C48: renamed from C49; value 10uF, 10V, 0805 -> 10uF
- C49: renamed from C50; value 0u1F, 10V, 0603 -> 0.1uF
- C50: renamed from C46; footprint Capacitor_SMD:C_0805_2012Metric_Pad1.18x1.45mm_HandSolder -> Capacitor_SMD:C_1206_3216Metric_Pad1.33x1.80mm_HandSolder
- D3: renamed from D4; value D -> LIN Diode
- D4: renamed from D3; value D -> LIN Diode
- IC3, IC4: Height 1.1 -> (none); Manufacturer_Name Texas Instruments -> (none); Manufacturer_Part_Number TLIN1039DDFRQ1 -> (none); Mouser Part Number 595-TLIN1039DDFRQ1 -> (none); Mouser Price/Stock https://www.mouser.co.uk/ProductDetail/Texas-Instruments/TL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 -> (none)
- J10: renamed from J8; value LIN-2 -> LIN CMD; now left out of the parts list
- J11: value LIN-2 -> LIN; MANUFACTURER Molex -> (none); MAXIMUM_PACKAGE_HEIGHT 3.5 mm -> (none); PARTREV A -> (none); STANDARD Manufacturer Recommendations -> (none)
- J8: renamed from J9; value LIN-1 -> LIN CMD; now left out of the parts list
- J9: renamed from J10; value LIN-1 -> LIN; MANUFACTURER Molex -> (none); MAXIMUM_PACKAGE_HEIGHT 3.5 mm -> (none); PARTREV A -> (none); STANDARD Manufacturer Recommendations -> (none)
- R22: renamed from R25; footprint Resistor_SMD:R_0805_2012Metric_Pad1.20x1.40mm_HandSolder -> Resistor_SMD:R_0603_1608Metric_Pad0.98x0.95mm_HandSolder
- R25: renamed from R24; footprint Resistor_SMD:R_0805_2012Metric_Pad1.20x1.40mm_HandSolder -> Resistor_SMD:R_0603_1608Metric_Pad0.98x0.95mm_HandSolder
- renumbered R22 to R24
Connections:
- net LIN1: now also TP23.1 (TP)
- net LIN1_EN: now also TP22.1 (TP)
- net LIN1_RX: now also TP20.1 (TP)
- net LIN1_TX: now also TP21.1 (TP)
- net LIN2: now also TP27.1 (TP)
- net LIN2_EN: now also TP26.1 (TP)
- net LIN2_RX: now also TP24.1 (TP)
- net LIN2_TX: now also TP25.1 (TP)
Other:
- note added: "Test Points LIN - 1"
- note added: "Test Points LIN - 2"
- note removed: "PWR LIN_2"

Commit message: new Design for Prototyping
Parts:
- removed J11, J9: LIN, 0530480210_2pin_P1.25_PicoBlade:MOLEX_530480210, symbol 0530480210_2pin_P1.25_PicoBlade:530480210
- added J10: LIN_2, TerminalBlock_Phoenix:TerminalBlock_Phoenix_PT-1,5-2-5.0-H_1x02_P5.00mm_Horizontal, symbol Connector:Screw_Terminal_01x02
- added J8: LIN_1, TerminalBlock_Phoenix:TerminalBlock_Phoenix_PT-1,5-2-5.0-H_1x02_P5.00mm_Horizontal, symbol Connector:Screw_Terminal_01x02
- renumbered C45 to C48, C46 to C49, C47 to C50, C48 to C51, C49 to C52, C50 to C53, IC3 to IC4, IC4 to IC5, J8 to J7, J10 to J9, R22 to R20, R23 to R21, R24 to R22, R25 to R23, TP20 to TP15, TP21 to TP16, TP22 to TP17, TP23 to TP18, TP24 to TP19, TP25 to TP20, TP26 to TP21, TP27 to TP22
Connections:
- net GND1: now also J10.2 (Pin_2), J8.2 (Pin_2)
- net LIN1: now also J8.1 (Pin_1)
- net LIN2: now also J10.1 (Pin_1)
Other:
- title: Rapid-Core -> (none)
- moved on the sheet: C51, C52, C53, D4, IC5, J9, R22, R23
