File: Design/General.kicad_sch (KiCad schematic)
At the start: 7 parts, among them J2 GPIO_CONN_X_4, J3 SPI, J4 USART, J5 SWD_Debug, SW1 SW_Push

Commit message: Layout complete
Parts:
- C30: value 0u1F -> 0.1uF
- J2: renamed from J5; now left out of the parts list
- J3: renamed from J2; now left out of the parts list
- J4: now left out of the parts list
- J5: renamed from J3; now left out of the parts list

Commit message: new Design for Prototyping
Parts:
- removed J3: GPIO_CONN_X_4, Connector_PinHeader_2.54mm:PinHeader_1x06_P2.54mm_Vertical, symbol Connector:Conn_01x06_Pin
- removed J4: USART, Connector_PinHeader_2.54mm:PinHeader_1x04_P2.54mm_Vertical, symbol Connector:Conn_01x04_Pin
- removed J5: SPI, Connector_PinHeader_2.54mm:PinHeader_1x05_P2.54mm_Vertical, symbol Connector:Conn_01x05_Pin
- added J4: USART, Connector_PinHeader_2.54mm:PinHeader_1x06_P2.54mm_Vertical, symbol Connector:Conn_01x06_Pin
- added J5: Conn_01x20_Pin, Connector_PinHeader_2.54mm:PinHeader_1x20_P2.54mm_Vertical, symbol Connector:Conn_01x20_Pin
- renumbered C30 to C33, J2 to J6, R9 to R7
Connections:
- net +3.3V: now also J4.1 (Pin_1)
- net GND1: now also J4.5 (Pin_5), J4.6 (Pin_6), J5.3 (Pin_3)
- net NRST: now also J6.4 (Pin_4); no longer J6.3 (Pin_3)
- net SPI1_MISO: now also J5.19 (Pin_19)
- net SPI1_MOSI: now also J5.18 (Pin_18)
- net SPI1_SCK: now also J5.20 (Pin_20)
- net SWDIO: now also J6.3 (Pin_3); no longer J6.4 (Pin_4)
- new net ADC_INP4: J5.17 (Pin_17)
- new net ADC_INP5: J5.14 (Pin_14)
- new net ADC_INP8: J5.16 (Pin_16)
- new net ADC_INP9: J5.15 (Pin_15)
- new net GPIO_1: J5.13 (Pin_13)
- new net GPIO_10: J5.4 (Pin_4)
- new net GPIO_2: J5.12 (Pin_12)
- new net GPIO_3: J5.11 (Pin_11)
- new net GPIO_4: J5.10 (Pin_10)
- new net GPIO_5: J5.9 (Pin_9)
- new net GPIO_6: J5.8 (Pin_8)
- new net GPIO_7: J5.7 (Pin_7)
- new net GPIO_8: J5.6 (Pin_6)
- new net GPIO_9: J5.5 (Pin_5)
- new net I2C_SCL_1: J5.2 (Pin_2)
- new net I2C_SDA_1: J5.1 (Pin_1)
- new net USART_CLK: J4.2 (Pin_2)
- new net USART_RX: J4.3 (Pin_3)
- new net USART_TX: J4.4 (Pin_4)
Other:
- note added: "External GPIO/I2C_1/SPI_1/ADC"
- note added: "External USART/UART/I2C"
- note removed: "External SPI"
- note removed: "External USART/UART"
- note removed: "GPIO Pins"
- title: Rapid-Core -> (none)
- moved on the sheet: C33, J6, R7, SW1
