File: Design/Indication - USR.kicad_sch (KiCad schematic)
At the start: 12 parts, among them Q1 NMOS, Q2 NMOS

Commit message: Layout complete
Parts:
- renumbered D10 to D7, D9 to D8, D7 to D9, Q2 to Q1, Q1 to Q2, R47 to R44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

Commit message: new Design for Prototyping
Parts:
- renumbered R44 to R42, R45 to R43, R46 to R44, R47 to R45, R48 to R46, R49 to R47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
Other:
- title: Rapid-Core -> (none)
- moved on the sheet: D9, R48
