File: Design/MCU.kicad_sch (KiCad schematic)
At the start: 21 parts, among them U4 STM32F446RETx, Y1 32.768_KHz, Y2 Crystal_GND24

Commit message: Layout complete
Parts:
- removed TP4, TP5: TestPoint, TestPoint:TestPoint_Pad_D1.0mm, symbol Connector:TestPoint
- C13: renamed from C26; value 0.1uf -> 0.1uF
- C14: renamed from C13; value 20pF, 0603 -> 20pF
- C15: renamed from C18; value 10uf -> 10uF
- C16: renamed from C21; value 1uf -> 1uF
- C17: renamed from C23; value 0.1uf -> 0.1uF
- C19: renamed from C15; value 15pf -> 15pF
- C20: renamed from C17; value 10uf -> 10uF
- C21: renamed from C19; value 1uf -> 1uF
- C22: renamed from C20; value 0.1uf -> 0.1uF
- C23: renamed from C22; value 0.1uf -> 0.1uF
- C24, C25: value 0.1uf -> 0.1uF
- C27: value 4.7uf 6.3V XR7 -> 4.7uF 6.3V XR7
- renumbered C14 to C18, C16 to C26, Y2 to Y1, Y1 to Y2
Connections:
- net USR_LED_1: now also U4.14 (PA0); no longer U4.58 (PB6)
- net USR_LED_2: now also U4.15 (PA1); no longer U4.59 (PB7)

Commit message: new Design for Prototyping
Parts:
- removed U4: STM32F446RETx, Package_QFP:LQFP-64_10x10mm_P0.5mm, symbol MCU_ST_STM32F4:STM32F446RETx
- added C19, C28: 0.1uF 16V X7R, Capacitor_SMD:C_0603_1608Metric_Pad1.08x0.95mm_HandSolder, symbol Device:C
- added C29: 4.7uF 6.3V XR7, Capacitor_SMD:C_0805_2012Metric_Pad1.18x1.45mm_HandSolder, symbol Device:C
- added J2: HSE_SEL, Connector_PinHeader_2.54mm:PinHeader_1x03_P2.54mm_Vertical, symbol Connector:Conn_01x03_Pin
- added J3: BOOT_SEL, Connector_PinHeader_2.54mm:PinHeader_1x02_P2.54mm_Vertical, symbol Connector:Conn_01x02_Pin
- added U3: STM32H750VBTx, Package_QFP:LQFP-100_14x14mm_P0.5mm, symbol MCU_ST_STM32H7:STM32H750VBTx
- C13: renamed from C14; now not fitted
- C14: renamed from C13; value 0.1uF -> 0.1uF 16V X7R
- C15: value 10uF -> 10uF 16V X7R
- C16: value 1uF -> 1uF 16V X7R
- C17: value 0.1uF -> 0.1uF 16V X7R
- C18, Y1: now not fitted
- C22: renamed from C20; value 10uF -> 10uF 16V X7R
- C23: renamed from C21; value 1uF -> 1uF 16V X7R
- C24: renamed from C22; value 0.1uF -> 0.1uF 16V X7R
- C25: renamed from C23; value 0.1uF -> 0.1uF 16V X7R
- C26: renamed from C24; value 0.1uF -> 0.1uF 16V X7R
- C27: renamed from C25; value 0.1uF -> 0.1uF 16V X7R
- renumbered C19 to C20, C26 to C21, C27 to C30, R6 to R4
Connections:
- net +3.3V: now also C19.1, C28.1, J2.3 (Pin_3), U3.100 (VDD), U3.11 (VDD), U3.20 (VREF+), U3.21 (VDDA), U3.27 (VDD), U3.50 (VDD), U3.6 (VBAT), U3.75 (VDD)
- net BOOT0: now also J3.1 (Pin_1), U3.94 (BOOT0); no longer R4.1
- net CAN1_RX: now also U3.95 (PB8)
- net CAN1_TX: now also U3.96 (PB9)
- net CAN2_RX: now also U3.91 (PB5)
- net CAN2_TX: now also U3.92 (PB6)
- net GND1: now also C19.2, C28.2, C29.2, J2.1 (Pin_1), U3.10 (VSS), U3.19 (VSSA), U3.26 (VSS), U3.49 (VSS), U3.74 (VSS), U3.99 (VSS); no longer Y1.4
- net HSE_IN: now also Y1.1, U3.12 (PH0); no longer Y1.3
- net HSE_OUT: now also Y1.3, U3.13 (PH1); no longer Y1.1
- net I2C_SCL_HUM: now also U3.59 (PD12)
- net I2C_SDA_HUM: now also U3.60 (PD13)
- net LIN1_EN: now also U3.23 (PA1)
- net LIN1_RX: now also U3.25 (PA3)
- net LIN1_TX: now also U3.24 (PA2)
- net LIN2_EN: now also U3.70 (PA11)
- net LIN2_RX: now also U3.69 (PA10)
- net LIN2_TX: now also U3.68 (PA9)
- net NRST: now also U3.14 (NRST)
- net RCC_OSC_32_IN: now also U3.8 (PC14)
- net RCC_OSC_32_OUT: now also U3.9 (PC15)
- net RS-485_1_EN: now also U3.80 (PC12)
- net RS-485_1_RX: now also U3.79 (PC11)
- net RS-485_1_TX: now also U3.78 (PC10)
- net RS-485_2_EN: now also U3.88 (PD7)
- net RS-485_2_RX: now also U3.89 (PB3)
- net RS-485_2_TX: now also U3.90 (PB4)
- net SPI1_MISO: now also U3.30 (PA6)
- net SPI1_MOSI: now also U3.31 (PA7)
- net SPI1_SCK: now also U3.29 (PA5)
- net SWDIO: now also U3.72 (PA13)
- net SW_CLK: now also U3.76 (PA14)
- net USR_LED_1: now also U3.2 (PE3)
- net USR_LED_2: now also U3.3 (PE4)
- net VCAP: now also C29.1, U3.48 (VCAP), U3.73 (VCAP)
- new net ADC_INP4: U3.32 (PC4)
- new net ADC_INP5: U3.35 (PB1)
- new net ADC_INP8: U3.33 (PC5)
- new net ADC_INP9: U3.34 (PB0)
- new net BOOT_SEL: J3.2 (Pin_2), R4.1
- new net GPIO_1: U3.36 (PB2)
- new net GPIO_10: U3.45 (PE15)
- new net GPIO_2: U3.37 (PE7)
- new net GPIO_3: U3.38 (PE8)
- new net GPIO_4: U3.39 (PE9)
- new net GPIO_5: U3.40 (PE10)
- new net GPIO_6: U3.41 (PE11)
- new net GPIO_7: U3.42 (PE12)
- new net GPIO_8: U3.43 (PE13)
- new net GPIO_9: U3.44 (PE14)
- new net HSE_SEL: J2.2 (Pin_2), Y1.4
- new net I2C_SCL_1: U3.46 (PB10)
- new net I2C_SDA_1: U3.47 (PB11)
- new net SPI_HOLD_FLASH: U3.55 (PD8)
- new net SPI_MISO_FLASH: U3.53 (PB14)
- new net SPI_MOSI_FLASH: U3.54 (PB15)
- new net SPI_NSS/CS_FLASH: U3.51 (PB12)
- new net SPI_SCK_FLASH: U3.52 (PB13)
- new net SPI_WP_FLASH: U3.56 (PD9)
- new net USART_CLK: U3.65 (PC8)
- new net USART_RX: U3.64 (PC7)
- new net USART_TX: U3.63 (PC6)
- no-connect marks 15 -> 28
Other:
- note added: "CL21B106KOQNNNG"
- title: Rapid-Core -> (none)
- moved on the sheet: C14, C15, C16, C17, C20, C21, C22, C23, C24, C25, C26, C27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
