File: Design/Misc.kicad_sch (KiCad schematic)
At the start: 11 parts

Commit message: Layout complete
Parts:
- renumbered FID3 to FID2, FID2 to FID3, H3 to H2, H2 to H3

Commit message: new Design for Prototyping
Parts:
- removed FID1, FID2, FID3: Fiducial, Fiducial:Fiducial_1.5mm_Mask3mm, symbol Mechanical:Fiducial
- removed G1: Not_to_bin, Not_To_Bin:Not_To_Bin, symbol Not_To_Bin:Not_To_Bin
- removed G2: NOON_REAY_ENERGIES, Noon_Ray:Noon_Ray, symbol Noon_Ray:Noon_Ray
- removed G3: High_Voltage_Warning, High_Voltage_Warning_logo:High_Voltage_Warning, symbol High_Voltage_Warning:HIgh_Voltage_Warning
- removed G4: ESD_Protection, ESD_Protection_Sign:ESD_Protection_Sign, symbol ESD_protection_warning_sign:LOGO
- removed H1, H2, H3, H4: MountingHole_Pad, MountingHole:MountingHole_2.2mm_M2_Pad, symbol Mechanical:MountingHole_Pad
- added G1: NoonRay_Energies_Pvt_Ltd, Noon_Ray:Noon_Ray_Mid_sized, symbol Noon_Ray:LOGO
Other:
- note removed: "Fiducials"
- note removed: "Front"
- note removed: "Logo"
- note removed: "Mounting Holes"
- title: Rapid-Core -> (none)
