File: Design/Power - Generation.kicad_sch (KiCad schematic)
At the start: 26 parts, among them IC1 LM60440ARPKR, J14 XT60PW-F, U1 LP3963-3.3, U2 CRE1S0505S3C, U3 CRE1S0505S3C

Commit message: Layout complete
Parts:
- removed TP1, TP2, TP3: TestPoint, TestPoint:TestPoint_Pad_D1.0mm, symbol Connector:TestPoint
- added TP1, TP2, TP3, TP4, TP5: Test_point, Test_point:Test_point, symbol Test_point:Test_point
- added TP6, TP7, TP8, TP9: GND, TestPoint:TestPoint_Loop_D2.60mm_Drill1.6mm_Beaded, symbol Test_point:Test_point
- C1: renamed from C8; value 0.1uF 1m -> 0.1uF, 1mohm; Digi _key (none) -> ₹26.06; Element 14 (none) -> ----; Manufacturer (none) -> KEMET; Manufacturer Part No (none) -> C0603C104J5RACAUTO; Mouser (none) -> C0603C104J5RACAUTO; Price 1's (none) -> ₹8.34; Price 1's Digi (none) -> In stock; Price 1's Ele 14 (none) -> C0603C104J5RACAUTO; Price 10's (none) -> ₹5.42; Price 10's Digi (none) -> ₹40.36; Price 10's Ele 14 (none) -> In stock; Type (none) -> SMD/Front
- C10: renamed from C7; footprint Capacitor_SMD:C_0603_1608Metric_Pad1.08x0.95mm_HandSolder -> Capacitor_SMD:C_0805_2012Metric_Pad1.18x1.45mm_HandSolder
- C6: renamed from C10; footprint Capacitor_SMD:C_0805_2012Metric_Pad1.18x1.45mm_HandSolder -> Capacitor_SMD:C_1206_3216Metric_Pad1.33x1.80mm_HandSolder
- C7: renamed from C11; footprint Capacitor_SMD:C_0805_2012Metric_Pad1.18x1.45mm_HandSolder -> Capacitor_SMD:C_1206_3216Metric_Pad1.33x1.80mm_HandSolder
- C8: renamed from C12; footprint Capacitor_SMD:C_0805_2012Metric_Pad1.18x1.45mm_HandSolder -> Capacitor_SMD:C_1206_3216Metric_Pad1.33x1.80mm_HandSolder
- C9: renamed from C5; footprint Capacitor_SMD:C_0603_1608Metric_Pad1.08x0.95mm_HandSolder -> Capacitor_SMD:C_0805_2012Metric_Pad1.18x1.45mm_HandSolder
- IC1: Height 0.7 -> (none); Manufacturer_Name Texas Instruments -> (none); Manufacturer_Part_Number LM60440ARPKR -> (none); Mouser Part Number 595-LM60440ARPKR -> (none); Mouser Price/Stock https://www.mouser.co.uk/ProductDetail/Texas-Instruments/LM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 -> (none)
- J1: renamed from J14; MANUFACTURER AMASS -> (none)
- L1: MANUFACTURER PART NO  XAL6060-822MEC -> (none)
- R1: renamed from R4; footprint Resistor_SMD:R_0805_2012Metric_Pad1.20x1.40mm_HandSolder -> Resistor_SMD:R_0603_1608Metric_Pad0.98x0.95mm_HandSolder
- R2: renamed from R3; footprint Resistor_SMD:R_0805_2012Metric_Pad1.20x1.40mm_HandSolder -> Resistor_SMD:R_0603_1608Metric_Pad0.98x0.95mm_HandSolder
- R3: renamed from R5; footprint Resistor_SMD:R_0805_2012Metric_Pad1.20x1.40mm_HandSolder -> Resistor_SMD:R_0402_1005Metric_Pad0.72x0.64mm_HandSolder
- R4: renamed from R1; footprint Resistor_SMD:R_0805_2012Metric_Pad1.20x1.40mm_HandSolder -> Resistor_SMD:R_0603_1608Metric_Pad0.98x0.95mm_HandSolder
- R5: renamed from R2; footprint Resistor_SMD:R_0805_2012Metric_Pad1.20x1.40mm_HandSolder -> Resistor_SMD:R_0603_1608Metric_Pad0.98x0.95mm_HandSolder
- renumbered C1 to C11, C6 to C12, C9 to C5
Connections:
- net +24V is gone; now on net VBAT: C2.1, C3.1, C4.1, IC1.10 (VIN_2), IC1.2 (VIN_1), IC1.9 (EN)
- net +3.3V: now also TP3.1 (TP)
- net +5V: now also TP2.1 (TP)
- net +5VA: now also TP4.1 (TP), TP5.1 (TP)
- net GND1: now also TP7.1 (TP), TP8.1 (TP)
- net GND2: now also TP6.1 (TP), TP9.1 (TP)
- net VBAT: now also TP1.1 (TP)
Other:
- note added: "Test Points"

Commit message: new Design for Prototyping
Parts:
- removed C11: 66uF LDO, Capacitor_SMD:CP_Elec_5x5.8, symbol Device:C_Polarized_US
- removed C12: 33uF LDO, Capacitor_SMD:CP_Elec_4x5.8, symbol Device:C_Polarized_US
- removed J1: XT60PW-F, XT60PW-F_Connector:AMASS_XT60PW-F, symbol XT60PW-F_Connector:XT60PW-F
- removed L1: 8.2mH 24mohm, Inductor_SMD:L_Coilcraft_XAL6060-XXX, symbol Device:L
- removed R4, R5: 10k LDO, Resistor_SMD:R_0603_1608Metric_Pad0.98x0.95mm_HandSolder, symbol Device:R
- removed TP1: Test_point, Test_point:Test_point, symbol Test_point:Test_point
- removed U1: LP3963-3.3, Package_TO_SOT_SMD:TO-263-5_TabPin3, symbol Regulator_Linear:LP3963-3.3
- added C11, C12: 0.1uF,LDO, Capacitor_SMD:C_0603_1608Metric_Pad1.08x0.95mm_HandSolder, symbol Device:C
- added IC2: BD33HC5WEFJ-E2, BD33HC5WEFJ-E2_LDO:SOIC127P600X100-9N, symbol BD33HC5WEFJ-E2_LDO:BD33HC5WEFJ-E2
- added J1: IN, TerminalBlock_Phoenix:TerminalBlock_Phoenix_PT-1,5-2-5.0-H_1x02_P5.00mm_Horizontal, symbol Connector:Screw_Terminal_01x02
- added L1: SRP6060FA-8R2M, SRP6060FA-8R2M_Inductor:SRP6060FA8R2M, symbol SRP6060FA-8R2M:SRP6060FA-8R2M
- C3, C4: footprint Capacitor_SMD:C_0603_1608Metric_Pad1.08x0.95mm_HandSolder -> Capacitor_SMD:C_0805_2012Metric_Pad1.18x1.45mm_HandSolder
- R3: value 24.9k -> 24.9k, 50V; footprint Resistor_SMD:R_0402_1005Metric_Pad0.72x0.64mm_HandSolder -> Resistor_SMD:R_0603_1608Metric_Pad0.98x0.95mm_HandSolder
- renumbered TP2 to TP1, TP4 to TP2, TP5 to TP3, TP6 to TP4, TP7 to TP5, TP8 to TP6, TP9 to TP7, TP3 to TP8, U2 to U1, U3 to U2
Connections:
- net +3.3V: now also C12.1, IC2.1 (VO), IC2.2 (VO_S)
- net +5V: now also C11.1, IC2.5 (EN), IC2.8 (VCC), L1.2
- net GND1: now also C11.2, C12.2, IC2.3 (GND), IC2.4 (NC_1), IC2.6 (NC_2), IC2.7 (NC_3), IC2.9 (EP), J1.2 (Pin_2)
- net LM_SW: now also L1.1
- net VBAT: now also J1.1 (Pin_1)
Other:
- title: Rapid-Core -> (none)
- moved on the sheet: TP8, U1, U2
