File: Design/Sensing - Hum_Temp.kicad_sch (KiCad schematic)
At the start: 5 parts, among them IC2 SHT30A-DIS-B2.5KS

Commit message: Layout complete
Parts:
- added TP10, TP11: Test_point, Test_point:Test_point, symbol Test_point:Test_point
- IC2: Height 1 -> (none); Manufacturer_Name Sensirion -> (none); Manufacturer_Part_Number SHT30A-DIS-B2.5KS -> (none); Mouser Part Number 403-SHT30ADIS-B2.5KS -> (none); Mouser Price/Stock https://www.mouser.co.uk/ProductDetail/Sensirion/SHT30A-DIS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 -> (none)
Connections:
- net I2C_SCL_HUM: now also TP11.1 (TP)
- net I2C_SDA_HUM: now also TP10.1 (TP)
Other:
- note added: "Test Points"

Commit message: new Design for Prototyping
Parts:
- renumbered C28 to C31, C29 to C32, IC2 to IC3, R7 to R5, R8 to R6, TP11 to TP10, TP10 to TP9
Other:
- title: Rapid-Core -> (none)
Changed lines of the file:
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@@
 	(generator_version "8.0")
 	(paper "A4")
-	(title_block
-		(title "Rapid-Core")
-		(date "2024-09-09")
-		(rev "1.0.1")
-	)
 	(junction
 		(at 149.86 81.28)
@@
 		)
 	)
-	(text_box "Design Note:\nI2C Address : 0x44(Default)\nR3 ,R4 pull-up resistors  \n"
+	(text_box "Design Note:\nI2C Address : 0x44(Default)\n"
 		(exclude_from_sim no)
 		(at 139.7 93.98 0)
-		(size 30.48 13.97)
+		(size 30.48 7.62)
 		(stroke
 			(width 1)
@@
 	)
 	(hierarchical_label "I2C_SDA_HUM"
-		(shape input)
+		(shape bidirectional)
 		(at 177.8 77.47 0)
 		(fields_autoplaced yes)
@@
 		(on_board yes)
 		(dnp no)
-		(property "Reference" "#PWR053"
+		(property "Reference" "#PWR054"
 			(at 74.93 83.82 0)
 			(effects
@@
 			(project "Rapid_Core-RCP"
 				(path "/1a5d67a4-b410-4c7a-b64e-9e0193c8e6b4/31f15dcd-2d12-4b77-aa4d-ff69e9876080/3ad87c0f-dff9-44e1-9550-eb9919a331d1"
-					(reference "#PWR053")
+					(reference "#PWR054")
 					(unit 1)
 				)
@@
 		(on_board yes)
 		(dnp no)
-		(property "Reference" "#PWR049"
+		(property "Reference" "#PWR050"
 			(at 74.93 68.58 0)
 			(effects
@@
 			(project "Rapid_Core-RCP"
 				(path "/1a5d67a4-b410-4c7a-b64e-9e0193c8e6b4/31f15dcd-2d12-4b77-aa4d-ff69e9876080/3ad87c0f-dff9-44e1-9550-eb9919a331d1"
-					(reference "#PWR049")
+					(reference "#PWR050")
 					(unit 1)
 				)
@@
 		(dnp no)
 		(fields_autoplaced yes)
-		(property "Reference" "R7"
+		(property "Reference" "R5"
 			(at 143.51 69.85 0)
 			(effects
@@
 			(project "Rapid_Core-RCP"
 				(path "/1a5d67a4-b410-4c7a-b64e-9e0193c8e6b4/31f15dcd-2d12-4b77-aa4d-ff69e9876080/3ad87c0f-dff9-44e1-9550-eb9919a331d1"
-					(reference "R7")
+					(reference "R5")
 					(unit 1)
 				)
@@
 		(on_board yes)
 		(dnp no)
-		(property "Reference" "#PWR055"
+		(property "Reference" "#PWR056"
 			(at 121.92 105.41 0)
 			(effects
@@
 			(project "Rapid_Core-RCP"
 				(path "/1a5d67a4-b410-4c7a-b64e-9e0193c8e6b4/31f15dcd-2d12-4b77-aa4d-ff69e9876080/3ad87c0f-dff9-44e1-9550-eb9919a331d1"
-					(reference "#PWR055")
+					(reference "#PWR056")
 					(unit 1)
 				)
@@
 		(dnp no)
 		(fields_autoplaced yes)
-		(property "Reference" "R8"
+		(property "Reference" "R6"
 			(at 152.4 69.85 0)
 			(effects
@@
 			(project "Rapid_Core-RCP"
 				(path "/1a5d67a4-b410-4c7a-b64e-9e0193c8e6b4/31f15dcd-2d12-4b77-aa4d-ff69e9876080/3ad87c0f-dff9-44e1-9550-eb9919a331d1"
-					(reference "R8")
+					(reference "R6")
 					(unit 1)
 				)
@@
 		(on_board yes)
 		(dnp no)
-		(property "Reference" "C29"
+		(property "Reference" "C32"
 			(at 86.36 68.58 0)
 			(effects
@@
 			(project "Rapid_Core-RCP"
 				(path "/1a5d67a4-b410-4c7a-b64e-9e0193c8e6b4/31f15dcd-2d12-4b77-aa4d-ff69e9876080/3ad87c0f-dff9-44e1-9550-eb9919a331d1"
-					(reference "C29")
+					(reference "C32")
 					(unit 1)
 				)
@@
 		(on_board yes)
 		(dnp no)
-		(property "Reference" "#PWR054"
+		(property "Reference" "#PWR055"
 			(at 104.14 99.06 0)
 			(effects
@@
 			(project "Rapid_Core-RCP"
 				(path "/1a5d67a4-b410-4c7a-b64e-9e0193c8e6b4/31f15dcd-2d12-4b77-aa4d-ff69e9876080/3ad87c0f-dff9-44e1-9550-eb9919a331d1"
-					(reference "#PWR054")
+					(reference "#PWR055")
 					(unit 1)
 				)
@@
 		(on_board yes)
 		(dnp no)
-		(property "Reference" "#PWR051"
+		(property "Reference" "#PWR052"
 			(at 149.86 69.85 0)
 			(effects
@@
 			(project "Rapid_Core-RCP"
 				(path "/1a5d67a4-b410-4c7a-b64e-9e0193c8e6b4/31f15dcd-2d12-4b77-aa4d-ff69e9876080/3ad87c0f-dff9-44e1-9550-eb9919a331d1"
-					(reference "#PWR051")
+					(reference "#PWR052")
 					(unit 1)
 				)
@@
 		(on_board yes)
 		(dnp no)
-		(property "Reference" "#PWR050"
+		(property "Reference" "#PWR051"
 			(at 140.97 69.85 0)
 			(effects
@@
 			(project "Rapid_Core-RCP"
 				(path "/1a5d67a4-b410-4c7a-b64e-9e0193c8e6b4/31f15dcd-2d12-4b77-aa4d-ff69e9876080/3ad87c0f-dff9-44e1-9550-eb9919a331d1"
-					(reference "#PWR050")
+					(reference "#PWR051")
 					(unit 1)
 				)
@@
 		(on_board yes)
 		(dnp no)
-		(property "Reference" "TP10"
+		(property "Reference" "TP9"
 			(at 76.962 168.148 90)
 			(effects
@@
 			(project "Rapid_Core-RCP"
 				(path "/1a5d67a4-b410-4c7a-b64e-9e0193c8e6b4/31f15dcd-2d12-4b77-aa4d-ff69e9876080/3ad87c0f-dff9-44e1-9550-eb9919a331d1"
-					(reference "TP10")
+					(reference "TP9")
 					(unit 1)
 				)
@@
 		(on_board yes)
 		(dnp no)
-		(property "Reference" "#PWR052"
+		(property "Reference" "#PWR053"
 			(at 121.92 72.39 0)
 			(effects
@@
 			(project "Rapid_Core-RCP"
 				(path "/1a5d67a4-b410-4c7a-b64e-9e0193c8e6b4/31f15dcd-2d12-4b77-aa4d-ff69e9876080/3ad87c0f-dff9-44e1-9550-eb9919a331d1"
-					(reference "#PWR052")
+					(reference "#PWR053")
 					(unit 1)
 				)
@@
 		(on_board yes)
 		(dnp no)
-		(property "Reference" "IC2"
+		(property "Reference" "IC3"
 			(at 124.1141 68.58 0)
 			(effects
@@
 			(project "Rapid_Core-RCP"
 				(path "/1a5d67a4-b410-4c7a-b64e-9e0193c8e6b4/31f15dcd-2d12-4b77-aa4d-ff69e9876080/3ad87c0f-dff9-44e1-9550-eb9919a331d1"
-					(reference "IC2")
+					(reference "IC3")
 					(unit 1)
 				)
@@
 		(on_board yes)
 		(dnp no)
-		(property "Reference" "C28"
+		(property "Reference" "C31"
 			(at 74.93 68.58 0)
 			(effects
@@
 			(project "Rapid_Core-RCP"
 				(path "/1a5d67a4-b410-4c7a-b64e-9e0193c8e6b4/31f15dcd-2d12-4b77-aa4d-ff69e9876080/3ad87c0f-dff9-44e1-9550-eb9919a331d1"
-					(reference "C28")
+					(reference "C31")
 					(unit 1)
 				)
@@
 		(on_board yes)
 		(dnp no)
-		(property "Reference" "TP11"
+		(property "Reference" "TP10"
 			(at 77.216 171.45 90)
 			(effects
@@
 			(project "Rapid_Core-RCP"
 				(path "/1a5d67a4-b410-4c7a-b64e-9e0193c8e6b4/31f15dcd-2d12-4b77-aa4d-ff69e9876080/3ad87c0f-dff9-44e1-9550-eb9919a331d1"
-					(reference "TP11")
+					(reference "TP10")
 					(unit 1)
 				)
